File: reflow_station.kicad_sch (KiCad schematic)
At the start: 247 parts, among them IC1 AMC23C10DWVR, IC2 MP100LGN-Z, J1 F52Q-1A7H1-11015, J4 USB_A, M1 Fan_CPU_4pin, M2 Fan_CPU_4pin, M3 Fan_CPU_4pin, M4 Fan_CPU_4pin, P1 IEC_60320_C13_Plug, Q1 BTA16-600B, SW1 SW_DPST_x2, U1 TPS82130, U10 RCLAMP0504F.TCT, U5 MOC3023M, U6 ADS1118IDGS, U7 ADS1118IDGS, U9 TPS2051BDBVR

Commit message: feat: connect mcu pins and usb-uart (cdc)
Parts:
- removed C? (x2): 47p, symbol Device:C
- removed C? (x3): 100n, symbol Device:C
- removed C?: 4.7u, symbol Device:C
- removed D? (x2): LED, symbol Device:LED
- removed R? (x2): 27, symbol Device:R
- removed R? (x2): 330, Resistor_SMD:R_0402_1005Metric, symbol Device:R
- removed SW? (x2): SW_SPST, symbol Switch:SW_SPST
- removed TP? (x4): TestPoint, symbol Connector:TestPoint
- removed U?: FT230XQ, Package_DFN_QFN:QFN-16-1EP_4x4mm_P0.65mm_EP2.1x2.1mm, symbol Interface_USB:FT230XQ
- added R? (x4): 10k, symbol Device:R
- added SW? (x2): SW_SPST, symbol Switch:SW_SPST
- added TP? (x4): TestPoint, symbol Connector:TestPoint
- F1, P1, SW1: now left out of the parts list
- R41: value 47k -> 10k
- R?: value 10k -> 82k
- R?: value 4.7k -> 33k
Connections:
- net BOTTOM_HEATER_A is gone; now on net HEATER_C#: TP?.1, U?.2
- net BOTTOM_HEATER_B is gone; now on net HEATER_D#: TP?.1, U?.2
- net BOTTOM_TRIAC_A_ON is gone; now on net TRIAC_C_ON#: R?.2, SW?.3
- net BOTTOM_TRIAC_B_ON is gone; now on net TRIAC_D_ON#: R?.2, SW?.4
- net SCL0 is gone; now on net LCD_SCL: R?.1, TP?.1
- net SDA0 is gone; now on net LCD_SDA: R?.1, TP?.1
- net SPI_TH1_MISO is gone; now on net SPI_TC1_MISO: TP?.1, U6.9 (DOUT/~{DRDY})
- net SPI_TH1_MOSI is gone; now on net SPI_TC1_MOSI: TP?.1, U6.10 (DIN)
- net SPI_TH2_CLK is gone; now on net SPI_TC2_CLK: TP?.1, U7.1 (SCLK)
- net SPI_TH2_MISO is gone; now on net SPI_TC2_MISO: TP?.1, U7.9 (DOUT/~{DRDY})
- net SPI_TH2_MOSI is gone; now on net SPI_TC2_MOSI: TP?.1, U7.10 (DIN)
- net TOP_HEATER_A is gone; now on net HEATER_A#: TP?.1, U?.2
- net TOP_HEATER_B is gone; now on net HEATER_B#: TP?.1, U5.2
- net TOP_TRIAC_A_ON is gone; now on net TRIAC_A_ON#: R?.2, SW?.1
- net TOP_TRIAC_B_ON is gone; now on net TRIAC_B_ON#: R?.2, SW?.2
- net VBUS_SENSE is gone; now on net USB_UART_VBUS_SENSE: R?.1, R?.2
- net +3V3: now also D?.2 (A), D?.2 (A), D?.2 (A), D?.2 (A), D?.2 (A), D?.2 (A), R?.1, R?.1, R?.1
- net +5V: now also R?.2
- net AC_SYNC: now also U?.19 (PA0), U?.21 (PA2), U?.27 (PA6), U?.95 (PB6)
- net FANS_IN_TACHO: now also U?.71 (PA9)
- net FANS_OUT_TACHO: now also U?.67 (PC7)
- net GND: now also SW?.2 (B), SW?.2 (B), SW?.2 (B); no longer D?.1 (K), D?.1 (K), D?.1 (K), D?.1 (K), D?.1 (K), D?.1 (K)
- net SWO: no longer U?.92 (PB3)
- net USB_D+: now also U?.74 (PA12)
- net USB_D-: now also U?.73 (PA11)
- net USER_IN1#: now reaches R?.2, SW?.5
- net USER_IN1#: now also U?.39 (PE14)
- net USB_UART_D+: now reaches J?.A6 (D+), U?.6
- net USB_UART_D+: now also J?.B6 (D+), U?.49 (PB15)
- net USB_UART_D-: now reaches J?.A7 (D-), U?.1
- net USB_UART_D-: now also J?.B7 (D-), U?.48 (PB14)
- net USB_OC#: now reaches R41.1, U9.3 (~{OC})
- net DIODE_HEAT#: now reaches R?.1
- net DIODE_HEAT#: now also U?.86 (PD2)
- net at R?.2: now also D?.1 (K); no longer D?.2 (A) (x6)
- net DIODE_TEST#: now reaches R?.1
- net DIODE_TEST#: now also U?.89 (PD5)
- net DIODE_RUN#: now reaches R?.1
- net DIODE_RUN#: now also U?.84 (PD0)
- net RUN#: now reaches SW?.1 (A)
- net RUN#: now also U?.33 (PE8), R?.2
- net USER_IN4#: now reaches R?.2, SW?.8
- net USER_IN4#: now also U?.42 (PB11)
- net DIODE_FAIL#: now reaches R?.1
- net DIODE_FAIL#: now also U?.88 (PD4)
- net USER_IN2#: now reaches R?.2, SW?.6
- net USER_IN2#: now also U?.40 (PE15)
- net USER_IN3#: now reaches R?.2, SW?.7
- net USER_IN3#: now also U?.41 (PB10)
- net HEATER_A#: now reaches U?.20 (PA1)
- net HEATER_A#: now also TP?.1
- net HEATER_B#: now reaches U?.22 (PA3)
- net HEATER_B#: now also TP?.1
- net HEATER_C#: now reaches U?.28 (PA7)
- net HEATER_C#: now also TP?.1
- net KILL#: now reaches U?.32 (PE7)
- net KILL#: now also R?.2, SW?.1 (A)
- net STOP#: now reaches U?.34 (PE9)
- net STOP#: now also R?.2, SW?.1 (A)
- net TRIAC_A_ON#: now reaches U?.35 (PE10)
- net TRIAC_B_ON#: now reaches U?.36 (PE11)
- net TRIAC_C_ON#: now reaches U?.37 (PE12)
- net TRIAC_D_ON#: now reaches U?.38 (PE13)
- net USB_UART_VBUS_SENSE: now reaches U?.47 (PB13)
- net LCD_SDA: now reaches U?.69 (PC9)
- net LCD_SCL: now reaches U?.70 (PA8)
- net SPI_TC2_CLK: now reaches U?.81 (PC10)
- net SPI_TC2_MISO: now reaches U?.82 (PC11)
- net SPI_TC2_MOSI: now reaches U?.83 (PC12)
- net DIODE_STOP#: now reaches U?.85 (PD1)
- net DIODE_STOP#: now also R?.1
- net DIODE_COOL#: now reaches U?.87 (PD3)
- net DIODE_COOL#: now also R?.1
- net SPI_TC1_MISO: now reaches U?.93 (PB4)
- net SPI_TC1_MOSI: now reaches U?.94 (PB5)
- net HEATER_D#: now reaches U?.96 (PB7)
- net HEATER_D#: now also TP?.1
- net RESET renamed RESET#
- net SPI_TH1_CLK renamed SPI_TC1_CLK
- net SPI_TC1_CLK: now also U?.92 (PB3)
- net USB_EN renamed USB_EN#
- net USB_EN#: now also R?.1
- no-connect marks 13 -> 9
Other:
- moved on the sheet: C1, C19, C20, C21, C22, C23, C24, C25, C26, C38, C39, C4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

Commit message: feat: add "filter" to heaters and separate shield from GND
Parts:
- added C12: C, symbol Device:C
- added J1: 1731734, reflow_station_library:1731734, symbol reflow_station_symbols:1731734
- added L1: L, symbol Device:L
- added LS1: PS1240P02BT, reflow_station_library:PS1240P02BT, symbol reflow_station_symbols:PS1240P02BT
- added Q5: KSC1815YTA, Connector_PinHeader_1.00mm:PinHeader_1x03_P1.00mm_Vertical, symbol Simulation_SPICE:NPN
- added R46: 1k, symbol Device:R
- added R57: 470k, symbol Device:R
- IC1: footprint SOIC127P1150X280-8N -> reflow_station_library:SOIC127P1150X280-8N
- U10: renamed from U9; footprint DBV0005A_N -> reflow_station_library:DBV0005A_N
- gave numbers to parts that had none: 128
- renumbered C13 to C14, C14 to C15, C15 to C16, C17 to C18, C18 to C19, C4 to C2, C32 to C20, C33 to C21, C34 to C22, C35 to C23, C36 to C24, C37 to C25, C40 to C26, C41 to C27, C42 to C28, C43 to C29, C5 to C3, C44 to C30, C45 to C31, C46 to C32, C47 to C33, C48 to C34, C49 to C35, C19 to C36, C20 to C37, C21 to C38, C22 to C39, C2 to C4, C23 to C40, C24 to C41, C25 to C42, C26 to C43, C50 to C45, C51 to C46, C52 to C47, C3 to C5, C38 to C50, C39 to C51, C53 to C57, C54 to C58, D2 to D1, D1 to D2, J1 to J2, J4 to J3, Q1 to Q2, R17 to R12, R7 to R13, R20 to R14, R8 to R19, R9 to R20, R10 to R21, R11 to R22, R22 to R24, R23 to R26, R12 to R28, R13 to R29, R14 to R31, R15 to R32, R4 to R6, R25 to R62, R26 to R63, R27 to R64, R28 to R65, R29 to R66, R30 to R67, R31 to R68, R32 to R69, R5 to R7, R33 to R70, R34 to R71, R35 to R72, R36 to R73, R37 to R74, R38 to R75, R39 to R76, R40 to R77, R41 to R78, R6 to R8, U10 to U11, U5 to U4, U6 to U8, U7 to U9
Connections:
- net +3V3: now also LS1.1 (+), R46.2
- net Earth: now also J1.2
- net FANS_IN_PWM: now also U12.98 (PB8)
- net FANS_OUT_PWM: now also U12.99 (PB9)
- net GND: now also Q5.3 (E); no longer J2.MP1, J2.MP2, J2.MP3, J2.MP4, J3.SH (Shield), J4.SH (SHIELD), J5.9 (GNDDetect), U11.2, U13.2, U14.2
- net L: now also Q1.2 (A2); no longer R27.1
- net L_FUSED: now also J1.1; no longer F1.2
- net N: now also R27.1, C12.2, J1.3, L1.1; no longer SW1.2 (B)
- net at R27.2: now also C12.1, L1.2; no longer Q1.2 (A2)
- net BUZZER_ON: now reaches U12.26 (PA5)
- net BUZZER_ON: now also R57.1
- new net: LS1.2 (-), Q5.1 (C), R46.1
- new net: Q5.2 (B), R57.2
- new net L_FUSED_DNP: F1.2
- new net N_DNP: SW1.2 (B)
- new net SHIELD: J2.MP1, J2.MP2, J2.MP3, J2.MP4, J3.SH (Shield), J4.SH (SHIELD), J5.9 (GNDDetect), U11.2, U13.2, U14.2
- no-connect marks 9 -> 11
Other:
- note added: "230VAC power consumption: - +12V power consumption: 5.5W - Heaters power consumption: 4*1000W ------------------------------------ TOTAL: 4006W"
- note added: "Signaling"
- note removed: "230VAC power consumption: - +12V power consumption: 5.5W - Heaters power consumption: 3000W ------------------------------------ TOTAL: 3006W"
- note removed: "Bottom Heaters"
- note removed: "Signal Diodes"
- note removed: "Top Heaters"
- moved on the sheet: C1, C2, C3, D1, D10, D11, D6, D7, D8, D9, F1, P1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
