File: reflow_station.kicad_sch (KiCad schematic)
At the start: 245 parts, among them IC1 AMC23C10DWVR, IC2 MP100LGN-Z, J1 1731734, J2 F52Q-1A7H1-11015, J3 USB_A, J4 USB_C_Receptacle_USB2.0_16P, J5 Conn_ARM_JTAG_SWD_10, M1 Fan_CPU_4pin, M2 Fan_CPU_4pin, M3 Fan_CPU_4pin, M4 Fan_CPU_4pin, P1 IEC_60320_C13_Plug, Q1 BTA16-600B, Q2 BTA16-600B, Q3 BTA16-600B, Q4 BTA16-600B, Q5 KSC1815YTA, SW1 SW_DPST_x2, SW2 SW_DIP_x08, SW3 SW_SPST, SW4 SW_SPST, SW5 SW_SPST, SW6 SW_Push, SW7 SW_SPDT, SW8 SW_SPDT, U1 TPS82130, U10 TPS2051BDBVR, U11 RCLAMP0504F.TCT, U12 STM32F469VITx, U13 RCLAMP0504F.TCT, U14 RCLAMP0504F.TCT, U2 RAC20-12SK, U3 MOC3023M, U4 MOC3023M, U5 TPS82130, U6 MOC3023M, U7 MOC3023M, U8 ADS1118IDGS, U9 ADS1118IDGS, Y1 25MHz, Y2 32.768kHz

Commit message: feat: add footprints to symbols and extract symbol library
Parts:
- removed C12: C, symbol Device:C
- removed L1: L, symbol Device:L
- removed Q2, Q3, Q4: BTA16-600B, Package_TO_SOT_THT:TO-220-3_Vertical, symbol Triac_Thyristor:BTA16-600B
- removed R12, R25, R26, R35, R36, R41, R42: 220, symbol Device:R
- removed R14, R27, R37, R38: Heater, symbol Device:Heater
- removed TC1, TC2, TC3, TC4: Thermocouple, symbol Device:Thermocouple
- added C12, C13, C21, C22: 10n 305V X2, reflow_station_library:B32921C3103M000, symbol reflow_station_symbols:C
- added J10, J7, J8, J9: DG301-5.0-02P-12-00A_H_, reflow_station_library:DG3015002P1200AH, symbol reflow_station_symbols:DG301-5.0-02P-12-00A_H_
- added J2, J3, J5, J6: 1707027, reflow_station_library:1707027, symbol reflow_station_symbols:1707027
- added L2, L3, L4: 33R @ 100MHz, Inductor_SMD:L_1206_3216Metric_Pad1.22x1.90mm_HandSolder, symbol reflow_station_symbols:L
- added Q2, Q3, Q4: BTA16-600B, Package_TO_SOT_THT:TO-220-3_Vertical, symbol reflow_station_symbols:BTA16-600B
- added R12, R33, R34: 330 1W fusible, Resistor_THT:R_Axial_DIN0207_L6.3mm_D2.5mm_P10.16mm_Horizontal, symbol reflow_station_symbols:R
- added R18, R19, R35, R36: 33 0.5W, Resistor_SMD:R_0805_2012Metric_Pad1.20x1.40mm_HandSolder, symbol reflow_station_symbols:R
- added R75: 0, Resistor_SMD:R_0402_1005Metric, symbol reflow_station_symbols:R
- added RV1, RV2, RV3, RV4: 350VAC, Varistor:RV_Disc_D12mm_W3.9mm_P7.5mm, symbol reflow_station_symbols:Varistor
- C1, C2: symbol Device:C -> reflow_station_symbols:C
- C10, C6, C8: footprint (none) -> Capacitor_SMD:C_0402_1005Metric; symbol Device:C -> reflow_station_symbols:C
- C11: footprint (none) -> Capacitor_SMD:C_0603_1608Metric; symbol Device:C -> reflow_station_symbols:C
- C14: renamed from C13; footprint (none) -> Capacitor_SMD:C_1206_3216Metric_Pad1.33x1.80mm_HandSolder; symbol Device:C -> reflow_station_symbols:C
- C15: renamed from C14; footprint (none) -> Capacitor_SMD:C_1206_3216Metric; symbol Device:C -> reflow_station_symbols:C
- C16: renamed from C15; footprint (none) -> Capacitor_SMD:C_0603_1608Metric; symbol Device:C -> reflow_station_symbols:C
- C17: renamed from C16; footprint (none) -> Capacitor_SMD:CP_Elec_8x10.5; symbol Device:C_Polarized -> reflow_station_symbols:C_Polarized
- C18: renamed from C17; footprint (none) -> Capacitor_SMD:C_0402_1005Metric; symbol Device:C -> reflow_station_symbols:C
- C19: renamed from C18; footprint (none) -> Capacitor_SMD:C_0805_2012Metric; symbol Device:C_Polarized -> reflow_station_symbols:C
- C20: renamed from C19; footprint (none) -> Capacitor_SMD:C_0402_1005Metric; symbol Device:C -> reflow_station_symbols:C
- C23: renamed from C20; footprint (none) -> Capacitor_SMD:C_0402_1005Metric; symbol Device:C -> reflow_station_symbols:C
- C24: renamed from C21; footprint (none) -> Capacitor_SMD:C_0402_1005Metric; symbol Device:C -> reflow_station_symbols:C
- C25: renamed from C22; footprint (none) -> Capacitor_SMD:C_0805_2012Metric; symbol Device:C -> reflow_station_symbols:C
- C26: renamed from C23; footprint (none) -> Capacitor_SMD:C_0805_2012Metric; symbol Device:C -> reflow_station_symbols:C
- C27: renamed from C24; footprint (none) -> Capacitor_SMD:C_0402_1005Metric; symbol Device:C -> reflow_station_symbols:C
- C28: renamed from C25; footprint (none) -> Capacitor_SMD:C_0402_1005Metric; symbol Device:C -> reflow_station_symbols:C
- C29: renamed from C26; footprint (none) -> Capacitor_SMD:C_0402_1005Metric; symbol Device:C -> reflow_station_symbols:C
- C3: footprint (none) -> Capacitor_SMD:C_2220_5750Metric_Pad1.97x5.40mm_HandSolder; symbol Device:C -> reflow_station_symbols:C
- C30: renamed from C27; footprint (none) -> Capacitor_SMD:C_0402_1005Metric; symbol Device:C -> reflow_station_symbols:C
- C31: renamed from C28; footprint (none) -> Capacitor_SMD:C_0402_1005Metric; symbol Device:C -> reflow_station_symbols:C
- C32: renamed from C29; footprint (none) -> Capacitor_SMD:C_0402_1005Metric; symbol Device:C -> reflow_station_symbols:C
- C33: renamed from C30; footprint (none) -> Capacitor_SMD:C_0402_1005Metric; symbol Device:C -> reflow_station_symbols:C
- C34: renamed from C31; footprint (none) -> Capacitor_SMD:C_0402_1005Metric; symbol Device:C -> reflow_station_symbols:C
- C35: renamed from C32; footprint (none) -> Capacitor_SMD:C_0805_2012Metric; symbol Device:C -> reflow_station_symbols:C
- C36: renamed from C33; footprint (none) -> Capacitor_SMD:C_0805_2012Metric; symbol Device:C -> reflow_station_symbols:C
- C37: renamed from C34; footprint (none) -> Capacitor_SMD:C_0402_1005Metric; symbol Device:C -> reflow_station_symbols:C
- C38: renamed from C35; footprint (none) -> Capacitor_SMD:C_0402_1005Metric; symbol Device:C -> reflow_station_symbols:C
- C39: renamed from C36; footprint (none) -> Capacitor_SMD:C_0805_2012Metric; symbol Device:C -> reflow_station_symbols:C
- C4, C5: footprint (none) -> Capacitor_SMD:C_1206_3216Metric_Pad1.33x1.80mm_HandSolder; symbol Device:C -> reflow_station_symbols:C
- C40: renamed from C37; footprint (none) -> Capacitor_SMD:C_0402_1005Metric; symbol Device:C -> reflow_station_symbols:C
- C41: renamed from C38; footprint (none) -> Capacitor_SMD:C_0402_1005Metric; symbol Device:C -> reflow_station_symbols:C
- C42: renamed from C39; footprint (none) -> Capacitor_SMD:C_0402_1005Metric; symbol Device:C -> reflow_station_symbols:C
- C43: renamed from C40; footprint (none) -> Capacitor_SMD:C_0402_1005Metric; symbol Device:C -> reflow_station_symbols:C
- C44: renamed from C41; footprint (none) -> Capacitor_SMD:C_0402_1005Metric; symbol Device:C -> reflow_station_symbols:C
- C45: renamed from C42; footprint (none) -> Capacitor_SMD:C_0402_1005Metric; symbol Device:C -> reflow_station_symbols:C
- C46: renamed from C43; footprint (none) -> Capacitor_SMD:C_0402_1005Metric; symbol Device:C -> reflow_station_symbols:C
- C47: renamed from C44; footprint (none) -> Capacitor_SMD:C_0402_1005Metric; symbol Device:C -> reflow_station_symbols:C
- C48: renamed from C45; footprint (none) -> Capacitor_SMD:C_0402_1005Metric; symbol Device:C -> reflow_station_symbols:C
- C49: renamed from C46; footprint (none) -> Capacitor_SMD:C_0402_1005Metric; symbol Device:C -> reflow_station_symbols:C
- C50: renamed from C47; footprint (none) -> Capacitor_SMD:C_1206_3216Metric_Pad1.33x1.80mm_HandSolder; symbol Device:C -> reflow_station_symbols:C
- C51: renamed from C48; footprint (none) -> Capacitor_SMD:C_0402_1005Metric; symbol Device:C -> reflow_station_symbols:C
- C52: renamed from C49; footprint (none) -> Capacitor_SMD:C_0603_1608Metric; symbol Device:C -> reflow_station_symbols:C
- C53: renamed from C50; footprint (none) -> Capacitor_SMD:C_0402_1005Metric; symbol Device:C -> reflow_station_symbols:C
- C54: renamed from C51; footprint (none) -> Capacitor_SMD:C_0805_2012Metric; symbol Device:C -> reflow_station_symbols:C
- C55: renamed from C52; footprint (none) -> Capacitor_SMD:C_0402_1005Metric; symbol Device:C -> reflow_station_symbols:C
- C56: renamed from C53; footprint (none) -> Capacitor_SMD:C_0402_1005Metric; symbol Device:C -> reflow_station_symbols:C
- C57: renamed from C54; footprint (none) -> Capacitor_SMD:C_0805_2012Metric; symbol Device:C -> reflow_station_symbols:C
- C58: renamed from C55; footprint (none) -> Capacitor_SMD:C_0402_1005Metric; symbol Device:C -> reflow_station_symbols:C
- C59: renamed from C56; footprint (none) -> Capacitor_SMD:C_0402_1005Metric; symbol Device:C -> reflow_station_symbols:C
- C60: renamed from C57; footprint (none) -> Capacitor_SMD:C_0603_1608Metric; symbol Device:C -> reflow_station_symbols:C
- C61: renamed from C58; footprint (none) -> Capacitor_SMD:C_0603_1608Metric; symbol Device:C -> reflow_station_symbols:C
- C62: renamed from C59; footprint (none) -> Capacitor_SMD:C_0402_1005Metric; symbol Device:C -> reflow_station_symbols:C
- C63: renamed from C60; footprint (none) -> Capacitor_SMD:C_0402_1005Metric; symbol Device:C -> reflow_station_symbols:C
- C7, C9: footprint (none) -> Capacitor_SMD:C_0805_2012Metric; symbol Device:C -> reflow_station_symbols:C
- D1, D10, D2, D5, D7, D8: footprint (none) -> LED_SMD:LED_0603_1608Metric; symbol Device:LED -> reflow_station_symbols:LED
- D11, D6, D9: footprint (none) -> LED_SMD:LED_0805_2012Metric; symbol Device:LED -> reflow_station_symbols:LED
- D3: symbol Diode:BAT54S -> reflow_station_symbols:BAT54S
- D4: symbol Diode_Bridge:MBL110S -> reflow_station_symbols:MBL110S
- F1: symbol Device:Fuse -> reflow_station_symbols:Fuse
- J11: renamed from J3; footprint (none) -> Connector_USB:USB_A_Molex_67643_Horizontal; symbol Connector:USB_A -> reflow_station_symbols:USB_A
- J12: renamed from J4; footprint (none) -> GeT_Footprints_Library:USB-C_SMD-TYPE-C-31-M-12; symbol Connector:USB_C_Receptacle_USB2.0_16P -> reflow_station_symbols:USB_C_Receptacle_USB2.0_16P
- J13: renamed from J5; symbol Connector:Conn_ARM_JTAG_SWD_10 -> reflow_station_symbols:Conn_ARM_JTAG_SWD_10
- L1: renamed from L2; footprint (none) -> Inductor_SMD:L_0603_1608Metric; symbol Device:L -> reflow_station_symbols:L
- M1, M2, M3, M4: footprint (none) -> Connector_JST:JST_PH_S4B-PH-K_1x04_P2.00mm_Horizontal; symbol Motor:Fan_CPU_4pin -> reflow_station_symbols:Fan_CPU_4pin
- P1: symbol Connector:IEC_60320_C13_Plug -> reflow_station_symbols:IEC_60320_C13_Plug
- Q1: symbol Triac_Thyristor:BTA16-600B -> reflow_station_symbols:BTA16-600B
- Q5: symbol Simulation_SPICE:NPN -> reflow_station_symbols:NPN
- R1, R2: symbol Device:R -> reflow_station_symbols:R
- R10, R4, R5, R7, R8, R9: footprint (none) -> Resistor_SMD:R_0402_1005Metric; symbol Device:R -> reflow_station_symbols:R
- R11: value 220 -> 330 1W fusible; footprint (none) -> Resistor_THT:R_Axial_DIN0207_L6.3mm_D2.5mm_P10.16mm_Horizontal; symbol Device:R -> reflow_station_symbols:R
- R13: footprint (none) -> Resistor_SMD:R_0603_1608Metric; symbol Device:R -> reflow_station_symbols:R
- R14: renamed from R15; footprint (none) -> Resistor_SMD:R_0402_1005Metric; symbol Device:R -> reflow_station_symbols:R
- R15: renamed from R16; footprint (none) -> Resistor_SMD:R_0402_1005Metric; symbol Device:R -> reflow_station_symbols:R
- R16: renamed from R17; footprint (none) -> Resistor_SMD:R_0402_1005Metric; symbol Device:R -> reflow_station_symbols:R
- R17: renamed from R18; footprint (none) -> Resistor_SMD:R_0402_1005Metric; symbol Device:R -> reflow_station_symbols:R
- R20: renamed from R19; footprint (none) -> Resistor_SMD:R_1206_3216Metric_Pad1.30x1.75mm_HandSolder; symbol Device:R -> reflow_station_symbols:R
- R21: renamed from R20; footprint (none) -> Resistor_SMD:R_1206_3216Metric_Pad1.30x1.75mm_HandSolder; symbol Device:R -> reflow_station_symbols:R
- R22: renamed from R21; footprint (none) -> Resistor_SMD:R_1206_3216Metric_Pad1.30x1.75mm_HandSolder; symbol Device:R -> reflow_station_symbols:R
- R23: renamed from R22; footprint (none) -> Resistor_SMD:R_1206_3216Metric_Pad1.30x1.75mm_HandSolder; symbol Device:R -> reflow_station_symbols:R
- R24: renamed from R23; footprint (none) -> Resistor_SMD:R_0402_1005Metric; symbol Device:R -> reflow_station_symbols:R
- R25: renamed from R24; footprint (none) -> Resistor_SMD:R_0402_1005Metric; symbol Device:R -> reflow_station_symbols:R
- R26: renamed from R28; footprint (none) -> Resistor_SMD:R_0402_1005Metric; symbol Device:R -> reflow_station_symbols:R
- R27: renamed from R29; symbol Device:R -> reflow_station_symbols:R
- R28: renamed from R30; footprint (none) -> Resistor_SMD:R_0402_1005Metric; symbol Device:R -> reflow_station_symbols:R
- R29: renamed from R31; footprint (none) -> Resistor_SMD:R_0402_1005Metric; symbol Device:R -> reflow_station_symbols:R
- R3: footprint (none) -> Resistor_SMD:R_0805_2012Metric_Pad1.20x1.40mm_HandSolder; symbol Device:R -> reflow_station_symbols:R
- R30: renamed from R32; footprint (none) -> Resistor_SMD:R_0402_1005Metric; symbol Device:R -> reflow_station_symbols:R
- R31: renamed from R33; footprint (none) -> Resistor_SMD:R_0402_1005Metric; symbol Device:R -> reflow_station_symbols:R
- R32: renamed from R34; footprint (none) -> Resistor_SMD:R_0402_1005Metric; symbol Device:R -> reflow_station_symbols:R
- R37: renamed from R39; footprint (none) -> Resistor_SMD:R_0402_1005Metric; symbol Device:R -> reflow_station_symbols:R
- R38: renamed from R40; footprint (none) -> Resistor_SMD:R_0402_1005Metric; symbol Device:R -> reflow_station_symbols:R
- R39: renamed from R43; footprint (none) -> Resistor_SMD:R_0402_1005Metric; symbol Device:R -> reflow_station_symbols:R
- R40: renamed from R44; footprint (none) -> Resistor_SMD:R_0402_1005Metric; symbol Device:R -> reflow_station_symbols:R
- R41: renamed from R45; footprint (none) -> Resistor_SMD:R_0402_1005Metric; symbol Device:R -> reflow_station_symbols:R
- R42: renamed from R46; footprint (none) -> Resistor_SMD:R_0402_1005Metric; symbol Device:R -> reflow_station_symbols:R
- R43: renamed from R47; footprint (none) -> Resistor_SMD:R_0402_1005Metric; symbol Device:R -> reflow_station_symbols:R
- R44: renamed from R48; footprint (none) -> Resistor_SMD:R_0402_1005Metric; symbol Device:R -> reflow_station_symbols:R
- R45: renamed from R49; footprint (none) -> Resistor_SMD:R_0402_1005Metric; symbol Device:R -> reflow_station_symbols:R
- R46: renamed from R50; footprint (none) -> Resistor_SMD:R_0402_1005Metric; symbol Device:R -> reflow_station_symbols:R
- R47: renamed from R51; symbol Device:R -> reflow_station_symbols:R
- R48: renamed from R52; symbol Device:R -> reflow_station_symbols:R
- R49: renamed from R53; symbol Device:R -> reflow_station_symbols:R
- R50: renamed from R54; symbol Device:R -> reflow_station_symbols:R
- R51: renamed from R55; symbol Device:R -> reflow_station_symbols:R
- R52: renamed from R56; symbol Device:R -> reflow_station_symbols:R
- R53: renamed from R57; value 470k -> 47k; footprint (none) -> Resistor_SMD:R_0402_1005Metric; symbol Device:R -> reflow_station_symbols:R
- R54: renamed from R58; footprint (none) -> Resistor_SMD:R_0402_1005Metric; symbol Device:R -> reflow_station_symbols:R
- R55: renamed from R59; footprint (none) -> Resistor_SMD:R_0402_1005Metric; symbol Device:R -> reflow_station_symbols:R
- R56: renamed from R60; footprint (none) -> Resistor_SMD:R_0402_1005Metric; symbol Device:R -> reflow_station_symbols:R
- R57: renamed from R61; footprint (none) -> Resistor_SMD:R_0402_1005Metric; symbol Device:R -> reflow_station_symbols:R
- R58: renamed from R62; footprint (none) -> Resistor_SMD:R_0402_1005Metric; symbol Device:R -> reflow_station_symbols:R
- R59: renamed from R63; footprint (none) -> Resistor_SMD:R_0402_1005Metric; symbol Device:R -> reflow_station_symbols:R
- R6: footprint (none) -> Resistor_THT:R_Axial_DIN0922_L20.0mm_D9.0mm_P25.40mm_Horizontal; symbol Device:R -> reflow_station_symbols:R
- R60: renamed from R64; footprint (none) -> Resistor_SMD:R_0402_1005Metric; symbol Device:R -> reflow_station_symbols:R
- R61: renamed from R65; footprint (none) -> Resistor_SMD:R_0402_1005Metric; symbol Device:R -> reflow_station_symbols:R
- R62: renamed from R66; footprint (none) -> Resistor_SMD:R_0402_1005Metric; symbol Device:R -> reflow_station_symbols:R
- R63: renamed from R67; footprint (none) -> Resistor_SMD:R_0402_1005Metric; symbol Device:R -> reflow_station_symbols:R
- R64: renamed from R68; footprint (none) -> Resistor_SMD:R_0402_1005Metric; symbol Device:R -> reflow_station_symbols:R
- R65: renamed from R69; footprint (none) -> Resistor_SMD:R_0402_1005Metric; symbol Device:R -> reflow_station_symbols:R
- R66: renamed from R70; footprint (none) -> Resistor_SMD:R_0402_1005Metric; symbol Device:R -> reflow_station_symbols:R
- R67: renamed from R71; footprint (none) -> Resistor_SMD:R_0402_1005Metric; symbol Device:R -> reflow_station_symbols:R
- R68: renamed from R72; footprint (none) -> Resistor_SMD:R_0402_1005Metric; symbol Device:R -> reflow_station_symbols:R
- R69: renamed from R73; footprint (none) -> Resistor_SMD:R_0402_1005Metric; symbol Device:R -> reflow_station_symbols:R
- R70: renamed from R74; footprint (none) -> Resistor_SMD:R_0402_1005Metric; symbol Device:R -> reflow_station_symbols:R
- R71: renamed from R75; footprint (none) -> Resistor_SMD:R_0402_1005Metric; symbol Device:R -> reflow_station_symbols:R
- R72: renamed from R76; footprint (none) -> Resistor_SMD:R_0402_1005Metric; symbol Device:R -> reflow_station_symbols:R
- R73: renamed from R77; footprint (none) -> Resistor_SMD:R_0402_1005Metric; symbol Device:R -> reflow_station_symbols:R
- R74: renamed from R78; footprint (none) -> Resistor_SMD:R_0402_1005Metric; symbol Device:R -> reflow_station_symbols:R
- R76: renamed from R79; footprint (none) -> Resistor_SMD:R_0402_1005Metric; symbol Device:R -> reflow_station_symbols:R
- R77: renamed from R80; footprint (none) -> Resistor_SMD:R_0402_1005Metric; symbol Device:R -> reflow_station_symbols:R
- R78: renamed from R81; footprint (none) -> Resistor_SMD:R_0402_1005Metric; symbol Device:R -> reflow_station_symbols:R
- R79: renamed from R82; footprint (none) -> Resistor_SMD:R_0402_1005Metric; symbol Device:R -> reflow_station_symbols:R
- R80: renamed from R83; footprint (none) -> Resistor_SMD:R_0402_1005Metric; symbol Device:R -> reflow_station_symbols:R
- R81: renamed from R84; footprint (none) -> Resistor_SMD:R_0402_1005Metric; symbol Device:R -> reflow_station_symbols:R
- R82: renamed from R85; footprint (none) -> Resistor_SMD:R_0603_1608Metric; symbol Device:R -> reflow_station_symbols:R
- SW1: symbol Switch:SW_DPST_x2 -> reflow_station_symbols:SW_DPST_x2
- SW2: footprint (none) -> Button_Switch_THT:SW_DIP_SPSTx08_Slide_9.78x22.5mm_W7.62mm_P2.54mm; symbol Switch:SW_DIP_x08 -> reflow_station_symbols:SW_DIP_x08
- SW3, SW4, SW5: symbol Switch:SW_SPST -> reflow_station_symbols:SW_SPST
- SW6: footprint (none) -> GeT_Footprints_Library:SW_TS-1088-AR02016; symbol Switch:SW_Push -> reflow_station_symbols:SW_Push
- SW7, SW8: footprint (none) -> reflow_station_library:ESP1010; symbol Switch:SW_SPDT -> reflow_station_symbols:SW_SPDT_132
- TP1, TP10, TP11, TP12, TP13, TP14, TP15, TP16, TP17, TP18, TP19, TP2, TP20, TP21, TP22, TP23, TP24, TP25, TP26, TP27, TP28, TP29, TP3, TP30, TP31, TP32, TP33, TP34, TP35, TP36, TP37, TP38, TP39, TP4, TP40, TP5, TP6, TP7, TP8, TP9: footprint (none) -> TestPoint:TestPoint_Pad_D1.0mm; symbol Connector:TestPoint -> reflow_station_symbols:TestPoint
- U1, U5: symbol Converter_DCDC:TPS82130 -> reflow_station_symbols:TPS82130
- U12: symbol MCU_ST_STM32F4:STM32F469VITx -> reflow_station_symbols:STM32F469VITx
- U2: symbol Converter_ACDC:RAC20-12SK -> reflow_station_symbols:RAC20-12SK
- U3, U4, U6, U7: footprint (none) -> Package_DIP:DIP-6_W7.62mm_LongPads; symbol Relay_SolidState:MOC3023M -> reflow_station_symbols:MOC3023M
- U8, U9: symbol Analog_ADC:ADS1118IDGS -> reflow_station_symbols:ADS1118IDGS
- Y1: footprint (none) -> Crystal:Crystal_SMD_3225-4Pin_3.2x2.5mm; symbol Device:Crystal -> reflow_station_symbols:Crystal_GND24
- Y2: footprint (none) -> Crystal:Crystal_SMD_3215-2Pin_3.2x1.5mm; symbol Device:Crystal -> reflow_station_symbols:Crystal
- renumbered J2 to J4
Connections:
- net +3V3: now also SW7.2 (B), SW8.2 (B), R75.1; no longer C51.1, C52.1, SW7.3 (C), SW8.3 (C), U12.56 (VCAPDSI), U12.62 (VDD12DSI)
- net GND: now also Y1.2 (G), Y1.4 (G), L2.1, L3.1, L4.1
- net GND1: now also C11.2, D3.1 (A), D3.2 (K), IC1.3 (INN)
- net L: now also Q2.2 (A2), Q3.2 (A2), Q4.2 (A2), R12.2, R18.1, R19.1, R33.2, R34.2, R35.1, R36.1, RV1.1, RV2.1, RV3.1, RV4.1
- net N: now also J2.2, J3.2, J5.2, J6.2; no longer C11.2, D3.1 (A), D3.2 (K), IC1.3 (INN), Q1.1 (A1)
- net SHIELD: now also L2.2, L3.2, L4.2
- net at U4.6: now also R12.1
- net TC3-: now reaches R70.1, R72.2
- net TC3-: now also J9.2
- net TC3+: now reaches R66.1, R68.1
- net TC3+: now also J9.1
- net TC4+: now reaches R67.1, R69.1
- net TC4+: now also J10.1
- net at U6.6: now also R33.1
- net TC2+: now reaches R59.1, R61.1
- net TC2+: now also J8.1
- net TC2-: now reaches R63.1, R65.2
- net TC2-: now also J8.2
- net at Q1.3 (G): now also U3.4
- net at U7.4: now also Q4.3 (G)
- net at U7.6: now also R34.1
- net at C58.1, TP35.1, U12.9 (PH0): now also Y1.3; no longer Y1.2
- net TC4-: now reaches R71.1, R73.2
- net TC4-: now also J10.2
- net TC1-: now reaches R62.1, R64.2
- net TC1-: now also J7.2
- net TC1+: now reaches R58.1, R60.1
- net TC1+: now also J7.1
- net at R78.2: now also SW8.3 (C); no longer SW8.2 (B)
- net at U6.4: now also Q3.3 (G)
- net at U4.4: now also Q2.3 (G)
- net at R77.1: now also SW7.3 (C); no longer SW7.2 (B)
- new net: C13.2, J3.1, Q2.1 (A1), RV2.2
- new net: C12.1, R18.2
- new net: C21.2, J5.1, Q3.1 (A1), RV3.2
- new net: C12.2, J2.1, Q1.1 (A1), RV1.2
- new net: C21.1, R35.2
- new net: C22.1, R36.2
- new net: C22.2, J6.1, Q4.1 (A1), RV4.2
- new net: C13.1, R19.2
- new net VDD12DSI: C51.1, C52.1, R75.2, U12.56 (VCAPDSI), U12.62 (VDD12DSI)
Other:
- moved on the sheet: C10, C11, C58, C59, C9, IC1, Q1, R11, R13, R20, R21, R22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

Commit message: feat: update footprint library and assign 3d models
Parts:
- C1: footprint Capacitor_THT:C_Axial_L12.0mm_D6.5mm_P15.00mm_Horizontal -> reflow_station_library:C_Axial_L12.0mm_D6.5mm_P15.00mm_Horizontal; KiLib_Generator (none) -> capacitor/THT/other
- C10, C18, C20, C23, C24, C27, C28, C29, C30, C31, C32, C33, C34, C37, C38, C40, C41, C42, C43, C44, C45, C46, C47, C48, C49, C51, C53, C55, C56, C58, C59, C6, C62, C63, C8: footprint Capacitor_SMD:C_0402_1005Metric -> reflow_station_library:C_0402_1005Metric; KiLib_Generator (none) -> SMD_2terminal_chip_molded
- C11, C16, C52, C60, C61: footprint Capacitor_SMD:C_0603_1608Metric -> reflow_station_library:C_0603_1608Metric; KiLib_Generator (none) -> SMD_2terminal_chip_molded
- C14, C4, C5, C50: footprint Capacitor_SMD:C_1206_3216Metric_Pad1.33x1.80mm_HandSolder -> reflow_station_library:C_1206_3216Metric_Pad1.33x1.80mm_HandSolder; KiLib_Generator (none) -> SMD_2terminal_chip_molded
- C15: footprint Capacitor_SMD:C_1206_3216Metric -> reflow_station_library:C_1206_3216Metric; KiLib_Generator (none) -> SMD_2terminal_chip_molded
- C17: footprint Capacitor_SMD:CP_Elec_8x10.5 -> reflow_station_library:CP_Elec_8x10.5; KiLib_Generator (none) -> capacitor/SMD/elec_round_polarized
- C19, C25, C26, C35, C36, C39, C54, C57, C7, C9: footprint Capacitor_SMD:C_0805_2012Metric -> reflow_station_library:C_0805_2012Metric; KiLib_Generator (none) -> SMD_2terminal_chip_molded
- C2: footprint Capacitor_SMD:C_0603_1608Metric_Pad1.08x0.95mm_HandSolder -> reflow_station_library:C_0603_1608Metric_Pad1.08x0.95mm_HandSolder; KiLib_Generator (none) -> SMD_2terminal_chip_molded
- C3: footprint Capacitor_SMD:C_2220_5750Metric_Pad1.97x5.40mm_HandSolder -> reflow_station_library:C_2220_5750Metric_Pad1.97x5.40mm_HandSolder; KiLib_Generator (none) -> SMD_2terminal_chip_molded
- D1, D10, D2, D5, D7, D8: footprint LED_SMD:LED_0603_1608Metric -> reflow_station_library:LED_0603_1608Metric; KiLib_Generator (none) -> SMD_2terminal_chip_molded
- D11, D6, D9: footprint LED_SMD:LED_0805_2012Metric -> reflow_station_library:LED_0805_2012Metric; KiLib_Generator (none) -> SMD_2terminal_chip_molded
- D3: footprint Package_TO_SOT_SMD:SOT-23 -> reflow_station_library:SOT-23; KiLib_Generator (none) -> package/gullwing
- D4: JLC_3DModel (none) -> 6ef4e732a59e44bcbac362674dd9511b; JLC_3D_Size (none) -> 4.7 7
- J11: footprint Connector_USB:USB_A_Molex_67643_Horizontal -> reflow_station_library:USB_A_Molex_67643_Horizontal
- J12: footprint GeT_Footprints_Library:USB-C_SMD-TYPE-C-31-M-12 -> reflow_station_library:USB-C_SMD-TYPE-C-31-M-12
- J13: footprint Connector_PinHeader_1.27mm:PinHeader_2x05_P1.27mm_Vertical -> reflow_station_library:PinHeader_2x05_P1.27mm_Vertical; KiLib_Generator (none) -> connector/pin_header_socket
- L1: footprint Inductor_SMD:L_0603_1608Metric -> reflow_station_library:L_0603_1608Metric; KiLib_Generator (none) -> SMD_2terminal_chip_molded
- L2, L3, L4: footprint Inductor_SMD:L_1206_3216Metric_Pad1.22x1.90mm_HandSolder -> reflow_station_library:L_1206_3216Metric_Pad1.22x1.90mm_HandSolder; KiLib_Generator (none) -> SMD_2terminal_chip_molded
- M1, M2, M3, M4: footprint Connector_JST:JST_PH_S4B-PH-K_1x04_P2.00mm_Horizontal -> reflow_station_library:JST_PH_S4B-PH-K_1x04_P2.00mm_Horizontal; KiLib_Generator (none) -> connector/JST
- Q1, Q2, Q3, Q4: footprint Package_TO_SOT_THT:TO-220-3_Vertical -> reflow_station_library:TO-220-3_Vertical; KiLib_Generator (none) -> package/TO_SOT/THT
- Q5: footprint Connector_PinHeader_1.00mm:PinHeader_1x03_P1.00mm_Vertical -> reflow_station_library:PinHeader_1x03_P1.00mm_Vertical; KiLib_Generator (none) -> connector/pin_header_socket
- R1, R10, R14, R15, R16, R17, R2, R24, R25, R26, R27, R28, R29, R30, R31, R32, R37, R38, R39, R4, R40, R41, R42, R43, R44, R45, R46, R47, R48, R49, R5, R50, R51, R52, R53, R54, R55, R56, R57, R58, R59, R60, R61, R62, R63, R64, R65, R66, R67, R68, R69, R7, R70, R71, R72, R73, R74, R75, R76, R77, R78, R79, R8, R80, R81, R9: footprint Resistor_SMD:R_0402_1005Metric -> reflow_station_library:R_0402_1005Metric; KiLib_Generator (none) -> SMD_2terminal_chip_molded
- R11, R12, R33, R34: footprint Resistor_THT:R_Axial_DIN0207_L6.3mm_D2.5mm_P10.16mm_Horizontal -> reflow_station_library:R_Axial_DIN0207_L6.3mm_D2.5mm_P10.16mm_Horizontal; KiLib_Generator (none) -> resistor/THT
- R13, R82: footprint Resistor_SMD:R_0603_1608Metric -> reflow_station_library:R_0603_1608Metric; KiLib_Generator (none) -> SMD_2terminal_chip_molded
- R18, R19, R3, R35, R36: footprint Resistor_SMD:R_0805_2012Metric_Pad1.20x1.40mm_HandSolder -> reflow_station_library:R_0805_2012Metric_Pad1.20x1.40mm_HandSolder; KiLib_Generator (none) -> SMD_2terminal_chip_molded
- R20, R21, R22, R23: footprint Resistor_SMD:R_1206_3216Metric_Pad1.30x1.75mm_HandSolder -> reflow_station_library:R_1206_3216Metric_Pad1.30x1.75mm_HandSolder; KiLib_Generator (none) -> SMD_2terminal_chip_molded
- R6: footprint Resistor_THT:R_Axial_DIN0922_L20.0mm_D9.0mm_P25.40mm_Horizontal -> reflow_station_library:R_Axial_DIN0922_L20.0mm_D9.0mm_P25.40mm_Horizontal; KiLib_Generator (none) -> resistor/THT
- RV1, RV2, RV3, RV4: footprint Varistor:RV_Disc_D12mm_W3.9mm_P7.5mm -> reflow_station_library:RV_Disc_D12mm_W3.9mm_P7.5mm
- SW2: footprint Button_Switch_THT:SW_DIP_SPSTx08_Slide_9.78x22.5mm_W7.62mm_P2.54mm -> reflow_station_library:SW_DIP_SPSTx08_Slide_9.78x22.5mm_W7.62mm_P2.54mm; KiLib_Generator (none) -> button_switch/DIP
- SW3, SW4, SW5: footprint (none) -> reflow_station_library:JST_XH_B2B-XH-A_1x02_P2.50mm_Vertical; KiLib_Generator (none) -> connector/JST
- SW6: footprint GeT_Footprints_Library:SW_TS-1088-AR02016 -> reflow_station_library:SW_TS-1088-AR02016; Availability (none) -> Not in stock; Check_prices (none) -> https://www.snapeda.com/parts/TS-1088-AR02016/Xunpu/view-pa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; Description_1 (none) -> 50mA 4mm 100MΩ 100,000 Times 12V 160gf 3mm 2mm Round Button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; MANUFACTURER (none) -> Xunpu; MAXIMUM_PACKAGE_HEIGHT (none) -> 2.0 mm; MF (none) -> Xunpu; MP (none) -> TS-1088-AR02016; PARTREV (none) -> N/A; Package (none) -> Package; Price (none) -> None; STANDARD (none) -> Manufacturer Recommendations; SnapEDA_Link (none) -> https://www.snapeda.com/parts/TS-1088-AR02016/Xunpu/view-pa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
- TP1, TP10, TP11, TP12, TP13, TP14, TP15, TP16, TP17, TP18, TP19, TP2, TP20, TP21, TP22, TP23, TP24, TP25, TP26, TP27, TP28, TP29, TP3, TP30, TP31, TP32, TP33, TP34, TP35, TP36, TP37, TP38, TP39, TP4, TP40, TP5, TP6, TP7, TP8, TP9: footprint TestPoint:TestPoint_Pad_D1.0mm -> reflow_station_library:TestPoint_Pad_D1.0mm
- U1, U5: footprint Package_LGA:Texas_SIL0008D_MicroSiP-8-1EP_2.8x3mm_P0.65mm_EP1.1x1.9mm_ThermalVias -> reflow_station_library:Texas_SIL0008D_MicroSiP-8-1EP_2.8x3mm_P0.65mm_EP1.1x1.9mm_ThermalVias; KiLib_Generator (none) -> package/no_lead
- U12: footprint Package_QFP:LQFP-100_14x14mm_P0.5mm -> reflow_station_library:LQFP-100_14x14mm_P0.5mm; KiLib_Generator (none) -> package/gullwing
- U2: footprint Converter_ACDC:Converter_ACDC_Recom_RAC20-xxSK_THT -> reflow_station_library:Converter_ACDC_Recom_RAC20-xxSK_THT
- U3, U4, U6, U7: footprint Package_DIP:DIP-6_W7.62mm_LongPads -> reflow_station_library:DIP-6_W7.62mm_LongPads; KiLib_Generator (none) -> package/DIP/legacy
- U8, U9: footprint Package_SO:TSSOP-10_3x3mm_P0.5mm -> reflow_station_library:TSSOP-10_3x3mm_P0.5mm; KiLib_Generator (none) -> package/gullwing
- Y1: footprint Crystal:Crystal_SMD_3225-4Pin_3.2x2.5mm -> reflow_station_library:Crystal_SMD_3225-4Pin_3.2x2.5mm; KiLib_Generator (none) -> crystal_resonator_oscillator
- Y2: footprint Crystal:Crystal_SMD_3215-2Pin_3.2x1.5mm -> reflow_station_library:Crystal_SMD_3215-2Pin_3.2x1.5mm

Commit message: feat: populate elements on board
Parts:
- removed D4: MB10S, reflow_station_library:MBS_L4.7-W3.8-P2.40-LS7.0-TL, symbol reflow_station_symbols:MBL110S
- added D4: MB10S, reflow_station_library:MBS_L4.7-W3.8-P2.40-LS7.0-TL, symbol Diode_Bridge:MDB10S
- C1: footprint reflow_station_library:C_Axial_L12.0mm_D6.5mm_P15.00mm_Horizontal -> reflow_station_library:R474N31005001K
- R3: footprint reflow_station_library:R_0805_2012Metric_Pad1.20x1.40mm_HandSolder -> reflow_station_library:R_0402_1005Metric
Connections:
- net GND1: now also D4.2 (-)
- net L_FUSED: now also D4.3
- net L_RECTIFIED: now also D4.1 (+)
- net N: now also D4.4
Changed lines of the file:
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@@
 			)
 		)
-		(property "Footprint" "reflow_station_library:R_0805_2012Metric_Pad1.20x1.40mm_HandSolder"
+		(property "Footprint" "reflow_station_library:R_0402_1005Metric"
 			(at 305.562 57.15 90)
 			(hide yes)
@@
 	)
 	(symbol
-		(lib_id "reflow_station_symbols:MBL110S")
-		(at 52.07 113.03 0)
-		(unit 1)
-		(body_style 1)
-		(exclude_from_sim no)
-		(in_bom yes)
-		(on_board yes)
-		(in_pos_files yes)
-		(dnp no)
-		(fields_autoplaced yes)
-		(property "Reference" "D4"
-			(at 62.23 106.6098 0)
-			(show_name no)
-			(do_not_autoplace no)
-			(effects
-				(font
-					(size 1.27 1.27)
-				)
-			)
-		)
-		(property "Value" "MB10S"
-			(at 62.23 109.1498 0)
-			(show_name no)
-			(do_not_autoplace no)
-			(effects
-				(font
-					(size 1.27 1.27)
-				)
-			)
-		)
-		(property "Footprint" "reflow_station_library:MBS_L4.7-W3.8-P2.40-LS7.0-TL"
-			(at 55.88 109.855 0)
-			(hide yes)
-			(show_name no)
-			(do_not_autoplace no)
-			(effects
-				(font
-					(size 1.27 1.27)
-				)
-				(justify left)
-			)
-		)
-		(property "Datasheet" "http://www.vishay.com/docs/89959/mbl104s.pdf"
-			(at 52.07 113.03 0)
-			(hide yes)
-			(show_name no)
-			(do_not_autoplace no)
-			(effects
-				(font
-					(size 1.27 1.27)
-				)
-			)
-		)
-		(property "Description" "Miniature Glass Passivated Single-Phase Surface Mount Bridge Rectifiers, 700V Vrms, 1.0A If, MBLS SMD package"
-			(at 52.07 113.03 0)
-			(hide yes)
-			(show_name no)
-			(do_not_autoplace no)
-			(effects
-				(font
-					(size 1.27 1.27)
-				)
-			)
-		)
-		(property "JLC_3DModel" "6ef4e732a59e44bcbac362674dd9511b"
-			(at 52.07 113.03 0)
-			(hide yes)
-			(show_name no)
-			(do_not_autoplace no)
-			(effects
-				(font
-					(size 1.27 1.27)
-				)
-			)
-		)
-		(property "JLC_3D_Size" "4.7 7"
-			(at 52.07 113.03 0)
-			(hide yes)
-			(show_name no)
-			(do_not_autoplace no)
-			(effects
-				(font
-					(size 1.27 1.27)
-				)
-			)
-		)
-		(pin "3"
-		)
-		(pin "2"
-		)
-		(pin "4"
-		)
-		(pin "1"
-		)
-		(instances
-			(project "reflow_station"
-				(path "/77770e37-dda2-4cf3-b2f1-cea4793bc3be"
-					(reference "D4")
-					(unit 1)
-				)
-			)
-		)
-	)
-	(symbol
 		(lib_id "reflow_station_symbols:GNDA")
 		(at 165.1 396.24 0)
@@
 	)
 	(symbol
+		(lib_id "Diode_Bridge:MDB10S")
+		(at 52.07 113.03 0)
+		(unit 1)
+		(body_style 1)
+		(exclude_from_sim no)
+		(in_bom yes)
+		(on_board yes)
+		(in_pos_files yes)
+		(dnp no)
+		(fields_autoplaced yes)
+		(property "Reference" "D4"
+			(at 62.23 106.6098 0)
+			(show_name no)
+			(do_not_autoplace no)
+			(effects
+				(font
+					(size 1.27 1.27)
+				)
+			)
+		)
+		(property "Value" "MB10S"
+			(at 62.23 109.1498 0)
+			(show_name no)
+			(do_not_autoplace no)
+			(effects
+				(font
+					(size 1.27 1.27)
+				)
+			)
+		)
+		(property "Footprint" "reflow_station_library:MBS_L4.7-W3.8-P2.40-LS7.0-TL"
+			(at 52.07 113.03 0)
+			(hide yes)
+			(show_name no)
+			(do_not_autoplace no)
+			(effects
+				(font
+					(size 1.27 1.27)
+				)
+			)
+		)
+		(property "Datasheet" "https://www.onsemi.com/pub/Collateral/MDB8S-D.PDF"
+			(at 52.07 113.03 0)
+			(hide yes)
+			(show_name no)
+			(do_not_autoplace no)
+			(effects
+				(font
+					(size 1.27 1.27)
+				)
+			)
+		)
+		(property "Description" "Single-Phase Bridge Rectifier, 700V Vrms, 1A If, TSSOP-4"
+			(at 52.07 113.03 0)
+			(hide yes)
+			(show_name no)
+			(do_not_autoplace no)
+			(effects
+				(font
+					(size 1.27 1.27)
+				)
+			)
+		)
+		(pin "4"
+		)
+		(pin "1"
+		)
+		(pin "2"
+		)
+		(pin "3"
+		)
+		(instances
+			(project "reflow_station"
+				(path "/77770e37-dda2-4cf3-b2f1-cea4793bc3be"
+					(reference "D4")
+					(unit 1)
+				)
+			)
+		)
+	)
+	(symbol
 		(lib_id "reflow_station_symbols:R")
 		(at 831.85 549.91 90)
@@
 			)
 		)
-		(property "Footprint" "reflow_station_library:C_Axial_L12.0mm_D6.5mm_P15.00mm_Horizontal"
+		(property "Footprint" "reflow_station_library:R474N31005001K"
 			(at 130.5052 48.26 0)
 			(hide yes)

Commit message: feat: resize board; position elements more accurately; add mounting holes
Parts:
- added H1: MountingHole_Pad, MountingHole:MountingHole_3mm, symbol Mechanical:MountingHole
- added H2, H3, H4: MountingHole_Pad, MountingHole:MountingHole_3mm_Pad_Via, symbol Mechanical:MountingHole_Pad
- added HS1: Heatsink, symbol reflow_station_symbols:Heatsink
- D4: symbol Diode_Bridge:MDB10S -> reflow_station_symbols:MDB10S
- J13: footprint reflow_station_library:PinHeader_2x05_P1.27mm_Vertical -> reflow_station_library:CONN-TH_10P-P1.27_HX-JN1.27-2X5P-ZZ-H4.9
- M1, M2, M3, M4: footprint reflow_station_library:JST_PH_S4B-PH-K_1x04_P2.00mm_Horizontal -> Connector_JST:JST_PH_B4B-PH-K_1x04_P2.00mm_Vertical
- SW3, SW4, SW5: footprint reflow_station_library:JST_XH_B2B-XH-A_1x02_P2.50mm_Vertical -> Connector_JST:JST_PH_B2B-PH-K_1x02_P2.00mm_Vertical
Connections:
- net GND: now also H2.1
- net SHIELD: now also H3.1, H4.1
