File: reflow_station.kicad_sch (KiCad schematic)
At the start: 263 parts, among them IC1 AMC23C10DWVR, IC2 MP100LGN-Z, J1 1731734, J10 DG301-5.0-02P-12-00A_H_, J11 USB_A, J12 USB_C_Receptacle_USB2.0_16P, J13 Conn_ARM_JTAG_SWD_10, J2 1707027, J3 1707027, J4 F52Q-1A7H1-11015, J5 1707027, J6 1707027, J7 DG301-5.0-02P-12-00A_H_, J8 DG301-5.0-02P-12-00A_H_, J9 DG301-5.0-02P-12-00A_H_, M1 Fan_CPU_4pin, M2 Fan_CPU_4pin, M3 Fan_CPU_4pin, M4 Fan_CPU_4pin, P1 C20 Plug 20A, Q1 BTA16-600B, Q2 BTA16-600B, Q3 BTA16-600B, Q4 BTA16-600B, Q5 KSC1815YTA, SW1 SW_DPST_x2, SW2 SW_DIP_x08, SW3 SW_SPST, SW4 SW_SPST, SW5 SW_SPST, SW6 SW_Push, SW7 SW_SPDT, SW8 SW_SPDT, U1 TPS82130, U10 TPS2051BDBVR, U11 RCLAMP0504F.TCT, U12 STM32F469VIT6, U13 RCLAMP0504F.TCT, U14 RCLAMP0504F.TCT, U2 RAC20-12SK, U3 MOC3052M, U4 MOC3052M, U5 TPS82130, U6 MOC3052M, U7 MOC3052M, U8 ADS1118IDGS, U9 ADS1118IDGS, Y1 25MHz, Y2 32.768kHz

Commit message: feat: change flat schematic to hierarchical, change board dimensions and add keepout areas
Parts:
- removed C1: 100n 1kV, reflow_station_library:R474N31005001K, symbol reflow_station_symbols:C
- removed C10, C2, C20, C23, C24, C27, C28, C29, C30, C31, C33, C37, C38, C40, C41, C42, C43, C44, C45, C46, C47, C48, C49, C51, C53, C55, C56, C6: 100n, reflow_station_library:C_0402_1005Metric, symbol reflow_station_symbols:C
- removed C11: 2.2n, reflow_station_library:C_0603_1608Metric, symbol reflow_station_symbols:C
- removed C12, C13, C21, C22: 10n 305V X2, reflow_station_library:B32921C3103M000, symbol reflow_station_symbols:C
- removed C14, C4: 10u, reflow_station_library:C_1206_3216Metric_Pad1.33x1.80mm_HandSolder, symbol reflow_station_symbols:C
- removed C15: 22u, reflow_station_library:C_1206_3216Metric, symbol reflow_station_symbols:C
- removed C16: 470p, reflow_station_library:C_0603_1608Metric, symbol reflow_station_symbols:C
- removed C17: 220u, reflow_station_library:CP_Elec_8x10.5, symbol reflow_station_symbols:C_Polarized
- removed C18, C8: 430p, reflow_station_library:C_0402_1005Metric, symbol reflow_station_symbols:C
- removed C19, C39: 4.7u, reflow_station_library:C_0805_2012Metric, symbol reflow_station_symbols:C
- removed C25, C26, C35, C36, C54, C57, C7, C9: 1u, reflow_station_library:C_0805_2012Metric, symbol reflow_station_symbols:C
- removed C3: 47u, reflow_station_library:C_2220_5750Metric_Pad1.97x5.40mm_HandSolder, symbol reflow_station_symbols:C
- removed C32, C34: 10n, reflow_station_library:C_0402_1005Metric, symbol reflow_station_symbols:C
- removed C5, C50: 47u, reflow_station_library:C_1206_3216Metric_Pad1.33x1.80mm_HandSolder, symbol reflow_station_symbols:C
- removed C52, C60, C61: 2.2u, reflow_station_library:C_0603_1608Metric, symbol reflow_station_symbols:C
- removed C58, C59: 10p, reflow_station_library:C_0402_1005Metric, symbol reflow_station_symbols:C
- removed C62, C63: 1.5p, reflow_station_library:C_0402_1005Metric, symbol reflow_station_symbols:C
- removed D1, D10, D2, D5, D7, D8: LED, reflow_station_library:LED_0603_1608Metric, symbol reflow_station_symbols:LED
- removed D11, D6, D9: LED, reflow_station_library:LED_0805_2012Metric, symbol reflow_station_symbols:LED
- removed D3: BAT54S, reflow_station_library:SOT-23, symbol reflow_station_symbols:BAT54S
- removed D4: MB10S, reflow_station_library:SOP240P700X300-4N, symbol reflow_station_symbols:MDB10S
- removed HS1, HS2, HS3, HS4: Heatsink, reflow_station_library:Heatsink_Stonecold_HS-132_32x14mm_2xFixation1.5mm, symbol reflow_station_symbols:Heatsink
- removed IC1: AMC23C10DWVR, reflow_station_library:SOIC127P1150X280-8N, symbol reflow_station_symbols:AMC23C10DWVR
- removed IC2: MP100LGN-Z, reflow_station_library:SOIC127P600X170-9N, symbol reflow_station_symbols:MP100LGN-Z
- removed J1: 1731734, reflow_station_library:1731734, symbol reflow_station_symbols:1731734
- removed J10, J7, J8, J9: DG301-5.0-02P-12-00A_H_, reflow_station_library:DG3015002P1200AH, symbol reflow_station_symbols:DG301-5.0-02P-12-00A_H_
- removed J11: USB_A, reflow_station_library:USB_A_Molex_67643_Horizontal, symbol reflow_station_symbols:USB_A
- removed J12: USB_C_Receptacle_USB2.0_16P, reflow_station_library:USB-C_SMD-TYPE-C-31-M-12, symbol reflow_station_symbols:USB_C_Receptacle_USB2.0_16P
- removed J13: Conn_ARM_JTAG_SWD_10, reflow_station_library:CONN-TH_10P-P1.27_HX-JN1.27-2X5P-ZZ-H4.9, symbol reflow_station_symbols:Conn_ARM_JTAG_SWD_10
- removed J2, J3, J5, J6: 1707027, reflow_station_library:1731721, symbol reflow_station_symbols:1731721
- removed J4: F52Q-1A7H1-11015, reflow_station_library:F52Q1A7H111015, symbol reflow_station_symbols:F52Q-1A7H1-11015
- removed L1: 600R @ 100MHz, reflow_station_library:L_0603_1608Metric, symbol reflow_station_symbols:L
- removed L2, L3, L4: 33R @ 100MHz, reflow_station_library:L_1206_3216Metric_Pad1.22x1.90mm_HandSolder, symbol reflow_station_symbols:L
- removed LS1: PS1240P02BT, reflow_station_library:PS1240P02BT, symbol reflow_station_symbols:PS1240P02BT
- removed M1, M2, M3, M4: Fan_CPU_4pin, reflow_station_library:JST_PH_B4B-PH-K_1x04_P2.00mm_Vertical, symbol reflow_station_symbols:Fan_CPU_4pin
- removed Q1, Q2, Q3, Q4: BTA16-600B, reflow_station_library:TO-220-3_Vertical_Staggered, symbol reflow_station_symbols:BTA16-600B
- removed Q5: KSC1815YTA, reflow_station_library:TO-92L_Inline_Wide, symbol reflow_station_symbols:NPN
- removed R1, R42: 1k, reflow_station_library:R_0402_1005Metric, symbol reflow_station_symbols:R
- removed R10, R14, R15, R16, R17, R4, R5, R75, R9: 0, reflow_station_library:R_0402_1005Metric, symbol reflow_station_symbols:R
- removed R11, R12, R33, R34: 470 1W fusible, reflow_station_library:R_Axial_DIN0411_L9.9mm_D3.6mm_P15.24mm_Horizontal, symbol reflow_station_symbols:R
- removed R13: 10, reflow_station_library:R_0603_1608Metric, symbol reflow_station_symbols:R
- removed R18, R19, R35, R36: 33 0.5W, reflow_station_library:C_1210_3225Metric, symbol reflow_station_symbols:R
- removed R2: 510, reflow_station_library:R_0402_1005Metric, symbol reflow_station_symbols:R
- removed R20, R21, R22: 1.09M, reflow_station_library:R_1206_3216Metric_Pad1.30x1.75mm_HandSolder, symbol reflow_station_symbols:R
- removed R23: 10k, reflow_station_library:R_1206_3216Metric_Pad1.30x1.75mm_HandSolder, symbol reflow_station_symbols:R
- removed R24, R25, R37, R38: 680, reflow_station_library:R_0402_1005Metric, symbol reflow_station_symbols:R
- removed R26, R31, R32, R7, R8: 100k, reflow_station_library:R_0402_1005Metric, symbol reflow_station_symbols:R
- removed R27, R47, R48, R49, R50, R51, R52: 330, reflow_station_library:R_0402_1005Metric, symbol reflow_station_symbols:R
- removed R28: 309k, reflow_station_library:R_0402_1005Metric, symbol reflow_station_symbols:R
- removed R29: 90.9k, reflow_station_library:R_0402_1005Metric, symbol reflow_station_symbols:R
- removed R3: 523k, reflow_station_library:R_0402_1005Metric, symbol reflow_station_symbols:R
- removed R30: 10.2k, reflow_station_library:R_0402_1005Metric, symbol reflow_station_symbols:R
- removed R39, R40, R41, R43, R44, R45, R46, R54, R55, R56, R57, R74, R76, R77, R78: 10k, reflow_station_library:R_0402_1005Metric, symbol reflow_station_symbols:R
- removed R53: 47k, reflow_station_library:R_0402_1005Metric, symbol reflow_station_symbols:R
- removed R58, R59, R64, R65, R66, R67, R72, R73: 1M, reflow_station_library:R_0402_1005Metric, symbol reflow_station_symbols:R
- removed R6: 100 3W, reflow_station_library:R_Axial_DIN0516_L15.5mm_D5.0mm_P20.32mm_Horizontal, symbol reflow_station_symbols:R
- removed R60, R61, R62, R63, R68, R69, R70, R71: 500, reflow_station_library:R_0402_1005Metric, symbol reflow_station_symbols:R
- removed R79, R80: 5.1k, reflow_station_library:R_0402_1005Metric, symbol reflow_station_symbols:R
- removed R81: 33k, reflow_station_library:R_0402_1005Metric, symbol reflow_station_symbols:R
- removed R82: 82k, reflow_station_library:R_0603_1608Metric, symbol reflow_station_symbols:R
- removed RV1, RV2, RV3, RV4: 350VAC, reflow_station_library:RV_Disc_D12mm_W3.9mm_P7.5mm, symbol reflow_station_symbols:Varistor
- removed SW2: SW_DIP_x08, reflow_station_library:SW_DIP_SPSTx08_Slide_9.78x22.5mm_W7.62mm_P2.54mm, symbol reflow_station_symbols:SW_DIP_x08
- removed SW3, SW4, SW5: SW_SPST, reflow_station_library:JST_PH_B2B-PH-K_1x02_P2.00mm_Vertical, symbol reflow_station_symbols:SW_SPST
- removed SW6: SW_Push, reflow_station_library:SW_TS-1088-AR02016, symbol reflow_station_symbols:SW_Push
- removed SW7, SW8: SW_SPDT, reflow_station_library:ESP1010, symbol reflow_station_symbols:SW_SPDT_132
- removed TP1, TP10, TP11, TP12, TP13, TP14, TP15, TP16, TP17, TP18, TP19, TP2, TP20, TP21, TP22, TP23, TP24, TP25, TP26, TP27, TP28, TP29, TP3, TP30, TP31, TP32, TP33, TP34, TP35, TP36, TP37, TP38, TP39, TP4, TP40, TP5, TP6, TP7, TP8, TP9: TestPoint, reflow_station_library:TestPoint_Pad_D1.0mm, symbol reflow_station_symbols:TestPoint
- removed U1, U5: TPS82130, reflow_station_library:Texas_SIL0008D_MicroSiP-8-1EP_2.8x3mm_P0.65mm_EP1.1x1.9mm_ThermalVias, symbol reflow_station_symbols:TPS82130
- removed U10: TPS2051BDBVR, reflow_station_library:DBV0005A_N, symbol reflow_station_symbols:TPS2051BDBVR
- removed U11, U13, U14: RCLAMP0504F.TCT, reflow_station_library:SC70-6L_RCLAMP_SEM, symbol reflow_station_symbols:RCLAMP0504F.TCT
- removed U12: STM32F469VIT6, reflow_station_library:LQFP-100_14x14mm_P0.5mm, symbol reflow_station_symbols:STM32F469VITx
- removed U2: RAC20-12SK, reflow_station_library:Converter_ACDC_Recom_RAC20-xxSK_THT, symbol reflow_station_symbols:RAC20-12SK
- removed U3, U4, U6, U7: MOC3052M, reflow_station_library:SMDIP-6_W9.53mm, symbol reflow_station_symbols:MOC3052M
- removed U8, U9: ADS1118IDGS, reflow_station_library:TSSOP-10_3x3mm_P0.5mm, symbol reflow_station_symbols:ADS1118IDGS
- removed Y1: 25MHz, reflow_station_library:Crystal_SMD_3225-4Pin_3.2x2.5mm, symbol reflow_station_symbols:Crystal_GND24
- removed Y2: 32.768kHz, reflow_station_library:Crystal_SMD_3215-2Pin_3.2x1.5mm, symbol reflow_station_symbols:Crystal
- H1: footprint reflow_station_library:MountingHole_3mm -> reflow_station_library:MountingHole_3mm_Pad_Via; symbol reflow_station_symbols:MountingHole -> Mechanical:MountingHole_Pad
Connections:
- net Earth: now also H1.1; no longer H3.1, H4.1
- net L_FUSED_DNP renamed LINE
- net N_DNP renamed NEUT
- new net SHIELD: H3.1, H4.1
- no-connect marks 11 -> 0
Other:
- added sheet AC Synchronization (ac_sync.kicad_sch)
- added sheet Connectivity (connectivity.kicad_sch)
- added sheet Device Configuration (config.kicad_sch)
- added sheet Fans (fans.kicad_sch)
- added sheet Heaters (heaters.kicad_sch)
- added sheet MCU (mcu.kicad_sch)
- added sheet Power (power.kicad_sch)
- added sheet Thermocouples (thermocouples.kicad_sch)
- added sheet User Interface (ui.kicad_sch)
- note removed: "+12V power consumption: - +5V power consumption (500mA): 2.5W - +3.3V power consumption (600mA): 2.0W - Fans: ___W ----------------------------------------- TOTAL: 4.5W + Fans"
- note removed: "+3.3V power consumption: - LCD (363mA): 1.2W - MCU (270mA): 0.9W - LED TRIAC (15mA): 0.04W - Thermocoup (600uA): 0.001W"
- note removed: "+5V power consumption: - LED(PWR): 5mA - USB: 500mA"
- note removed: "230VAC power consumption: - +12V power consumption: 5.5W - Heaters power consumption: 4*1000W ------------------------------------ TOTAL: 4006W"
- note removed: "AC Synchronization"
- note removed: "Control Switches"
- note removed: "Cooling"
- note removed: "Core"
- note removed: "Failure"
- note removed: "Fans"
- note removed: "Fans In"
- note removed: "Fans Out"
- note removed: "Heaters"
- note removed: "Heating"
- note removed: "Kill"
- note removed: "LCD"
- note removed: "Power"
- note removed: "Run"
- note removed: "Run / Resume"
- note removed: "SWD"
- note removed: "Self Test"
- note removed: "Signaling"
- note removed: "Stop"
- note removed: "Stop & Hold"
- note removed: "Thermocouples"
- note removed: "USB"
- note removed: "USB - UART"
- moved on the sheet: H2

Commit message: feat: add ground and earth(shield) planes, add better - multi layer connection for AC mains connector
Connections:
- net SHIELD is gone; now on net Earth: H3.1, H4.1
Changed lines of the file:
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@@
 		(company "Artur Twardzik")
 	)
+	(junction
+		(at 38.1 154.94)
+		(diameter 0)
+		(color 0 0 0 0)
+	)
 	(wire
 		(pts
@@
 	(wire
 		(pts
+			(xy 38.1 154.94) (xy 50.8 154.94)
+		)
+		(stroke
+			(width 0)
+			(type default)
+		)
+	)
+	(wire
+		(pts
 			(xy 50.8 152.4) (xy 50.8 154.94)
 		)
@@
 	(wire
 		(pts
-			(xy 25.4 154.94) (xy 50.8 154.94)
+			(xy 25.4 154.94) (xy 38.1 154.94)
 		)
 		(stroke
@@
 		(pts
 			(xy 165.1 38.1) (xy 165.1 50.8)
+		)
+		(stroke
+			(width 0)
+			(type default)
+		)
+	)
+	(wire
+		(pts
+			(xy 38.1 154.94) (xy 38.1 157.48)
 		)
 		(stroke
@@
 	(label "N_IN"
 		(at 38.1 25.4 0)
-		(effects
-			(font
-				(size 1.27 1.27)
-			)
-			(justify left bottom)
-		)
-	)
-	(label "SHIELD"
-		(at 33.02 154.94 0)
 		(effects
 			(font
@@
 					(unit 1)
 				)
+			)
+		)
+	)
+	(symbol
+		(lib_id "reflow_station_symbols:Earth")
+		(at 38.1 157.48 0)
+		(mirror y)
+		(unit 1)
+		(body_style 1)
+		(exclude_from_sim no)
+		(in_bom yes)
+		(on_board yes)
+		(in_pos_files yes)
+		(dnp no)
+		(property "Reference" "#PWR0177"
+			(at 38.1 163.83 0)
+			(hide yes)
+			(show_name no)
+			(do_not_autoplace no)
+			(effects
+				(font
+					(size 1.27 1.27)
+				)
+			)
+		)
+		(property "Value" "Earth"
+			(at 38.1 162.56 0)
+			(show_name no)
+			(do_not_autoplace no)
+			(effects
+				(font
+					(size 1.27 1.27)
+				)
+			)
+		)
+		(property "Footprint" ""
+			(at 38.1 157.48 0)
+			(hide yes)
+			(show_name no)
+			(do_not_autoplace no)
+			(effects
+				(font
+					(size 1.27 1.27)
+				)
+			)
+		)
+		(property "Datasheet" ""
+			(at 38.1 157.48 0)
+			(hide yes)
+			(show_name no)
+			(do_not_autoplace no)
+			(effects
+				(font
+					(size 1.27 1.27)
+				)
+			)
+		)
+		(property "Description" "Power symbol creates a global label with name \"Earth\""
+			(at 38.1 157.48 0)
+			(hide yes)
+			(show_name no)
+			(do_not_autoplace no)
+			(effects
+				(font
+					(size 1.27 1.27)
+				)
+			)
+		)
+		(pin "1"
+		)
+		(instances
+			(project "reflow_station"
+				(path "/77770e37-dda2-4cf3-b2f1-cea4793bc3be"
+					(reference "#PWR0177")
+					(unit 1)
+				)
