File: reflow_station.kicad_pcb (KiCad board)
At the start: 6 copper layers, 170 x 100 mm, 260 parts, among them IC1 AMC23C10DWVR, IC2 MP100LGN-Z, J1 1731734, J10 DG301-5.0-02P-12-00A_H_, J11 USB_A, J12 USB_C_Receptacle_USB2.0_16P, J13 Conn_ARM_JTAG_SWD_10, J2 1707027, J3 1707027, J4 F52Q-1A7H1-11015, J5 1707027, J6 1707027, J7 DG301-5.0-02P-12-00A_H_, J8 DG301-5.0-02P-12-00A_H_, J9 DG301-5.0-02P-12-00A_H_, M1 Fan_CPU_4pin, M2 Fan_CPU_4pin, M3 Fan_CPU_4pin, M4 Fan_CPU_4pin, Q1 BTA16-600B, Q2 BTA16-600B, Q3 BTA16-600B, Q4 BTA16-600B, Q5 KSC1815YTA, SW2 SW_DIP_x08, SW3 SW_SPST, SW4 SW_SPST, SW5 SW_SPST, SW6 SW_Push, SW7 SW_SPDT, SW8 SW_SPDT, U1 TPS82130, U10 TPS2051BDBVR, U11 RCLAMP0504F.TCT, U12 STM32F469VIT6, U13 RCLAMP0504F.TCT, U14 RCLAMP0504F.TCT, U2 RAC20-12SK, U3 MOC3052M, U4 MOC3052M, U5 TPS82130, U6 MOC3052M, U7 MOC3052M, U8 ADS1118IDGS, U9 ADS1118IDGS, Y1 25MHz, Y2 32.768kHz

Commit message: feat: change flat schematic to hierarchical, change board dimensions and add keepout areas
Parts:
- added C64: 2.2u, reflow_station_library:C_0603_1608Metric, F.Cu at (-55.2, 84.8)
- added C65: 1.5p, reflow_station_library:C_0402_1005Metric, F.Cu at (-58.6, 83.5)
- added C66: 1.5p, reflow_station_library:C_0402_1005Metric, F.Cu at (-58.6, 85.4)
- added D12: LED, reflow_station_library:LED_0805_2012Metric, F.Cu at (-40.5, 98.9)
- added D13: LED, reflow_station_library:LED_0603_1608Metric, F.Cu at (-40.7, 109.9)
- added D14: LED, reflow_station_library:LED_0805_2012Metric, F.Cu at (-40.5, 101.9)
- added L5: 33R @ 100MHz, reflow_station_library:L_1206_3216Metric_Pad1.22x1.90mm_HandSolder, F.Cu at (-103.8, 110.8)
- added L6: 33R @ 100MHz, reflow_station_library:L_1206_3216Metric_Pad1.22x1.90mm_HandSolder, F.Cu at (-103.8, 114.3)
- added R83: 0, reflow_station_library:R_0402_1005Metric, F.Cu at (-54.0, 61.0)
- added R84: 10k, reflow_station_library:R_0402_1005Metric, F.Cu at (-54.0, 63.0)
- added R85: 10k, reflow_station_library:R_0402_1005Metric, F.Cu at (-54.0, 65.0)
- C10: value 100n -> 220u; footprint reflow_station_library:C_0402_1005Metric -> reflow_station_library:CP_Elec_8x10.5
- C11: value 2.2n -> 430p; footprint reflow_station_library:C_0603_1608Metric -> reflow_station_library:C_0402_1005Metric
- C12: value 10n 305V X2 -> 4.7u; footprint reflow_station_library:B32921C3103M000 -> reflow_station_library:C_0805_2012Metric
- C13: value 10n 305V X2 -> 100n; footprint reflow_station_library:B32921C3103M000 -> reflow_station_library:C_0402_1005Metric
- C14: value 10u -> 100n; footprint reflow_station_library:C_1206_3216Metric_Pad1.33x1.80mm_HandSolder -> reflow_station_library:C_0402_1005Metric
- C15: value 22u -> 1u; footprint reflow_station_library:C_1206_3216Metric -> reflow_station_library:C_0402_1005Metric
- C16: value 470p -> 1u; footprint reflow_station_library:C_0603_1608Metric -> reflow_station_library:C_0402_1005Metric
- C17: value 220u -> 100n; footprint reflow_station_library:CP_Elec_8x10.5 -> reflow_station_library:C_0402_1005Metric
- C18: value 430p -> 2.2n; footprint reflow_station_library:C_0402_1005Metric -> reflow_station_library:C_0603_1608Metric
- C19: value 4.7u -> 10n 305V X2; footprint reflow_station_library:C_0805_2012Metric -> reflow_station_library:B32921C3103M000
- C20: value 100n -> 10n 305V X2; footprint reflow_station_library:C_0402_1005Metric -> reflow_station_library:B32921C3103M000
- C24, C27, C42, C43, C44: value 100n -> 1u
- C25, C26, C36, C54: value 1u -> 100n; footprint reflow_station_library:C_0805_2012Metric -> reflow_station_library:C_0402_1005Metric
- C30, C38: value 100n -> 10n
- C32: value 10n -> 1u
- C34: value 10n -> 100n
- C35, C57: footprint reflow_station_library:C_0805_2012Metric -> reflow_station_library:C_0402_1005Metric
- C39: value 4.7u -> 100n; footprint reflow_station_library:C_0805_2012Metric -> reflow_station_library:C_0402_1005Metric
- C40: value 100n -> 47u; footprint reflow_station_library:C_0402_1005Metric -> reflow_station_library:C_1206_3216Metric_Pad1.33x1.80mm_HandSolder
- C45: value 100n -> 4.7u; footprint reflow_station_library:C_0402_1005Metric -> reflow_station_library:C_0805_2012Metric
- C50: value 47u -> 100n; footprint reflow_station_library:C_1206_3216Metric_Pad1.33x1.80mm_HandSolder -> reflow_station_library:C_0402_1005Metric
- C52: value 2.2u -> 100n; footprint reflow_station_library:C_0603_1608Metric -> reflow_station_library:C_0402_1005Metric
- C55: value 100n -> 2.2u; footprint reflow_station_library:C_0402_1005Metric -> reflow_station_library:C_0603_1608Metric
- C58, C59: value 10p -> 100n
- C6: value 100n -> 430p
- C60: value 2.2u -> 1u; footprint reflow_station_library:C_0603_1608Metric -> reflow_station_library:C_0402_1005Metric
- C61: value 2.2u -> 10p; footprint reflow_station_library:C_0603_1608Metric -> reflow_station_library:C_0402_1005Metric
- C62: value 1.5p -> 10p
- C63: value 1.5p -> 2.2u; footprint reflow_station_library:C_0402_1005Metric -> reflow_station_library:C_0603_1608Metric
- C7: value 1u -> 10u; footprint reflow_station_library:C_0805_2012Metric -> reflow_station_library:C_1206_3216Metric_Pad1.33x1.80mm_HandSolder
- C8: value 430p -> 22u; footprint reflow_station_library:C_0402_1005Metric -> reflow_station_library:C_1206_3216Metric
- C9: value 1u -> 470p; footprint reflow_station_library:C_0805_2012Metric -> reflow_station_library:C_0603_1608Metric
- D11: footprint reflow_station_library:LED_0805_2012Metric -> reflow_station_library:LED_0603_1608Metric
- D3: value BAT54S -> MB10S; footprint reflow_station_library:SOT-23 -> reflow_station_library:SOP240P700X300-4N
- D4: value MB10S -> LED; footprint reflow_station_library:SOP240P700X300-4N -> reflow_station_library:LED_0603_1608Metric
- D5: value LED -> BAT54S; footprint reflow_station_library:LED_0603_1608Metric -> reflow_station_library:SOT-23
- D6: value LED -> 1N4148WS; footprint reflow_station_library:LED_0805_2012Metric -> Diode_SMD:D_SOD-323
- D7, D8: value LED -> 1N4148WS; footprint reflow_station_library:LED_0603_1608Metric -> Diode_SMD:D_SOD-323
- H1: footprint reflow_station_library:MountingHole_3mm -> reflow_station_library:MountingHole_3mm_Pad_Via
- IC1: value AMC23C10DWVR -> MP100LGN-Z; footprint reflow_station_library:SOIC127P1150X280-8N -> reflow_station_library:SOIC127P600X170-9N
- IC2: value MP100LGN-Z -> AMC23C10DWVR; footprint reflow_station_library:SOIC127P600X170-9N -> reflow_station_library:SOIC127P1150X280-8N
- J10: value DG301-5.0-02P-12-00A_H_ -> USB_A; footprint reflow_station_library:DG3015002P1200AH -> reflow_station_library:USB_A_Molex_67643_Horizontal
- J11: value USB_A -> USB_C_Receptacle_USB2.0_16P; footprint reflow_station_library:USB_A_Molex_67643_Horizontal -> reflow_station_library:USB-C_SMD-TYPE-C-31-M-12
- J12: value USB_C_Receptacle_USB2.0_16P -> Conn_ARM_JTAG_SWD_10; footprint reflow_station_library:USB-C_SMD-TYPE-C-31-M-12 -> reflow_station_library:CONN-TH_10P-P1.27_HX-JN1.27-2X5P-ZZ-H4.9
- J13: value Conn_ARM_JTAG_SWD_10 -> F52Q-1A7H1-11015; footprint reflow_station_library:CONN-TH_10P-P1.27_HX-JN1.27-2X5P-ZZ-H4.9 -> reflow_station_library:F52Q1A7H111015
- J4: value F52Q-1A7H1-11015 -> 1707027; footprint reflow_station_library:F52Q1A7H111015 -> reflow_station_library:1731721
- J6: value 1707027 -> DG301-5.0-02P-12-00A_H_; footprint reflow_station_library:1731721 -> reflow_station_library:DG3015002P1200AH
- L1: value 600R @ 100MHz -> 33R @ 100MHz; footprint reflow_station_library:L_0603_1608Metric -> reflow_station_library:L_1206_3216Metric_Pad1.22x1.90mm_HandSolder
- L4: value 33R @ 100MHz -> 600R @ 100MHz; footprint reflow_station_library:L_1206_3216Metric_Pad1.22x1.90mm_HandSolder -> reflow_station_library:L_0603_1608Metric
- R10: value 0 -> 90.9k
- R11: value 470 1W fusible -> 10.2k; footprint reflow_station_library:R_Axial_DIN0411_L9.9mm_D3.6mm_P15.24mm_Horizontal -> reflow_station_library:R_0402_1005Metric
- R12: value 470 1W fusible -> 100k; footprint reflow_station_library:R_Axial_DIN0411_L9.9mm_D3.6mm_P15.24mm_Horizontal -> reflow_station_library:R_0402_1005Metric
- R13: value 10 -> 100k; footprint reflow_station_library:R_0603_1608Metric -> reflow_station_library:R_0402_1005Metric
- R14: value 0 -> 10; footprint reflow_station_library:R_0402_1005Metric -> reflow_station_library:R_0603_1608Metric
- R15, R16, R17: value 0 -> 1.09M; footprint reflow_station_library:R_0402_1005Metric -> reflow_station_library:R_1206_3216Metric_Pad1.30x1.75mm_HandSolder
- R18: value 33 0.5W -> 10k; footprint reflow_station_library:C_1210_3225Metric -> reflow_station_library:R_1206_3216Metric_Pad1.30x1.75mm_HandSolder
- R19: value 33 0.5W -> 680; footprint reflow_station_library:C_1210_3225Metric -> reflow_station_library:R_0402_1005Metric
- R20: value 1.09M -> 680; footprint reflow_station_library:R_1206_3216Metric_Pad1.30x1.75mm_HandSolder -> reflow_station_library:R_0402_1005Metric
- R21, R22: value 1.09M -> 470 1W fusible; footprint reflow_station_library:R_1206_3216Metric_Pad1.30x1.75mm_HandSolder -> reflow_station_library:R_Axial_DIN0411_L9.9mm_D3.6mm_P15.24mm_Horizontal
- R23: value 10k -> 33 0.5W; footprint reflow_station_library:R_1206_3216Metric_Pad1.30x1.75mm_HandSolder -> reflow_station_library:C_1210_3225Metric
- R24: value 680 -> 33 0.5W; footprint reflow_station_library:R_0402_1005Metric -> reflow_station_library:C_1210_3225Metric
- R26: value 100k -> 680
- R27: value 330 -> 470 1W fusible; footprint reflow_station_library:R_0402_1005Metric -> reflow_station_library:R_Axial_DIN0411_L9.9mm_D3.6mm_P15.24mm_Horizontal
- R28: value 309k -> 470 1W fusible; footprint reflow_station_library:R_0402_1005Metric -> reflow_station_library:R_Axial_DIN0411_L9.9mm_D3.6mm_P15.24mm_Horizontal
- R29: value 90.9k -> 33 0.5W; footprint reflow_station_library:R_0402_1005Metric -> reflow_station_library:C_1210_3225Metric
- R30: value 10.2k -> 33 0.5W; footprint reflow_station_library:R_0402_1005Metric -> reflow_station_library:C_1210_3225Metric
- R31, R32: value 100k -> 1M
- R33, R34: value 470 1W fusible -> 1M; footprint reflow_station_library:R_Axial_DIN0411_L9.9mm_D3.6mm_P15.24mm_Horizontal -> reflow_station_library:R_0402_1005Metric
- R35, R36: value 33 0.5W -> 500; footprint reflow_station_library:C_1210_3225Metric -> reflow_station_library:R_0402_1005Metric
- R37, R38: value 680 -> 500
- R39, R40, R41: value 10k -> 1M
- R4: value 0 -> 100 3W; footprint reflow_station_library:R_0402_1005Metric -> reflow_station_library:R_Axial_DIN0516_L15.5mm_D5.0mm_P20.32mm_Horizontal
- R42: value 1k -> 1M
- R43, R44, R45, R46: value 10k -> 500
- R47, R48: value 330 -> 10k
- R49, R50: value 330 -> 5.1k
- R5: value 0 -> 100k
- R51: value 330 -> 33k
- R52: value 330 -> 82k; footprint reflow_station_library:R_0402_1005Metric -> reflow_station_library:R_0603_1608Metric
- R53: value 47k -> 10k
- R58: value 1M -> 10k
- R59: value 1M -> 1k
- R6: value 100 3W -> 100k; footprint reflow_station_library:R_Axial_DIN0516_L15.5mm_D5.0mm_P20.32mm_Horizontal -> reflow_station_library:R_0402_1005Metric
- R60, R61, R62, R63: value 500 -> 330
- R64, R65: value 1M -> 330
- R66: value 1M -> 47k
- R67, R72, R73: value 1M -> 0
- R68, R69, R70, R71: value 500 -> 0
- R74: value 10k -> 0
- R75: value 0 -> 10k
- R79, R80: value 5.1k -> 10k
- R8: value 100k -> 330
- R81: value 33k -> 10k
- R82: value 82k -> 10k; footprint reflow_station_library:R_0603_1608Metric -> reflow_station_library:R_0402_1005Metric
- R9: value 0 -> 309k
- SW2: value SW_DIP_x08 -> SW_SPST; footprint reflow_station_library:SW_DIP_SPSTx08_Slide_9.78x22.5mm_W7.62mm_P2.54mm -> reflow_station_library:JST_PH_B2B-PH-K_1x02_P2.00mm_Vertical
- SW5: value SW_SPST -> SW_DIP_x08; footprint reflow_station_library:JST_PH_B2B-PH-K_1x02_P2.00mm_Vertical -> reflow_station_library:SW_DIP_SPSTx08_Slide_9.78x22.5mm_W7.62mm_P2.54mm
- TP1, TP10, TP11, TP12, TP13, TP14, TP15, TP16, TP17, TP18, TP19, TP2, TP20, TP21, TP22, TP23, TP24, TP25, TP26, TP27, TP28, TP29, TP3, TP30, TP31, TP32, TP33, TP34, TP35, TP36, TP37, TP38, TP39, TP4, TP40, TP5, TP6, TP7, TP8, TP9: moved to F.Cu
- U12: value STM32F469VIT6 -> RCLAMP0504F.TCT; footprint reflow_station_library:LQFP-100_14x14mm_P0.5mm -> reflow_station_library:SC70-6L_RCLAMP_SEM
- U14: value RCLAMP0504F.TCT -> STM32F469VIT6; footprint reflow_station_library:SC70-6L_RCLAMP_SEM -> reflow_station_library:LQFP-100_14x14mm_P0.5mm
- U3: value MOC3052M -> TPS82130; footprint reflow_station_library:SMDIP-6_W9.53mm -> reflow_station_library:Texas_SIL0008D_MicroSiP-8-1EP_2.8x3mm_P0.65mm_EP1.1x1.9mm_ThermalVias
- U4, U6, U7: value MOC3052M -> MOC3052
- U5: value TPS82130 -> MOC3052; footprint reflow_station_library:Texas_SIL0008D_MicroSiP-8-1EP_2.8x3mm_P0.65mm_EP1.1x1.9mm_ThermalVias -> reflow_station_library:SMDIP-6_W9.53mm
- moved TP26 447.7 mm to (-132.0, 16.8)
- moved TP27 446.3 mm to (-132.0, 19.8)
- moved TP28 445.0 mm to (-132.0, 22.9)
- moved TP29 443.8 mm to (-132.0, 25.9)
- moved TP25 418.8 mm to (-113.8, 86.9)
- moved TP33 402.6 mm to (-96.1, 113.7)
- moved TP31 402.5 mm to (-99.2, 113.7)
- moved TP1 402.4 mm to (-102.4, 56.0)
- moved TP30 402.4 mm to (-99.2, 110.6)
- moved TP2 401.4 mm to (-102.4, 59.1)
- moved TP3 400.5 mm to (-102.4, 62.1)
- moved TP4 399.7 mm to (-102.4, 65.2)
- moved TP34 399.5 mm to (-93.1, 110.6)
- moved TP32 399.4 mm to (-96.1, 110.6)
- moved TP35 399.4 mm to (-93.1, 113.7)
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Connections:
- C1 pad 2: /N -> LINE
- C10 pad 1: GND1 -> Net-(IC1-VB)
- C10 pad 2: Net-(IC1-VDD1) -> GND1
- C11 pad 1: Net-(IC1-INP) -> Net-(U3-SS/TR)
- C11 pad 2: GND1 -> GND
- C12 pad 1: Net-(C12-Pad1) -> /Power/+12V_ISOLATED
- C12 pad 2: Net-(Q1-A1) -> GND1
- C13 pad 1: Net-(C13-Pad1) -> /Power/+12V_ISOLATED
- C13 pad 2: Net-(Q2-A1) -> GND1
- C14 pad 1: +12V -> +3V3
- C16 pad 1: Net-(IC2-FB) -> GND1
- C16 pad 2: /+12V_ISOLATED -> Net-(IC2-VDD1)
- C17 pad 1: Net-(IC2-VB) -> GND1
- C17 pad 2: GND1 -> Net-(IC2-VDD1)
- C18 pad 1: Net-(U5-SS/TR) -> Net-(IC2-INP)
- C18 pad 2: GND -> GND1
- C19 pad 1: /+12V_ISOLATED -> Net-(C19-Pad1)
- C19 pad 2: GND1 -> Net-(Q1-A1)
- C20 pad 1: /+12V_ISOLATED -> Net-(C20-Pad1)
- C20 pad 2: GND1 -> Net-(Q2-A1)
- C24 pad 1: GND -> Net-(U8-AIN0)
- C24 pad 2: Net-(U9-AIN0) -> Net-(U8-AIN1)
- C25 pad 1: Net-(U8-AIN0) -> Net-(U8-AIN1)
- C25 pad 2: Net-(U8-AIN1) -> GND
- C26 pad 1: Net-(U9-AIN0) -> GND
- C26 pad 2: Net-(U9-AIN1) -> Net-(U8-AIN2)
- C27 pad 1: Net-(U8-AIN1) -> Net-(U8-AIN2)
- C27 pad 2: GND -> Net-(U8-AIN3)
- C28 pad 1: Net-(U9-AIN1) -> Net-(U8-AIN3)
- C29 pad 1: GND -> +5V
- C29 pad 2: Net-(U8-AIN2) -> GND
- C30 pad 1: GND -> +5V
- C30 pad 2: Net-(U9-AIN2) -> GND
- C31 pad 1: +5V -> GND
- C31 pad 2: GND -> Net-(U9-AIN0)
- C32 pad 1: +5V -> Net-(U9-AIN0)
- C32 pad 2: GND -> Net-(U9-AIN1)
- C33 pad 1: +5V -> Net-(U9-AIN1)
- C34 pad 1: +5V -> GND
- C34 pad 2: GND -> Net-(U9-AIN2)
- C35 pad 1: Net-(U8-AIN2) -> Net-(U9-AIN2)
- C35 pad 2: Net-(U8-AIN3) -> Net-(U9-AIN3)
- C36 pad 1: Net-(U9-AIN2) -> Net-(U9-AIN3)
- C36 pad 2: Net-(U9-AIN3) -> GND
- C37 pad 1: Net-(U8-AIN3) -> +5V
- C38 pad 1: Net-(U9-AIN3) -> +5V
- C39 pad 1: +3V3 -> Net-(J10-VBUS)
- C40 pad 1: +3V3 -> Net-(J10-VBUS)
- C41 pad 1: +3V3 -> +5V
- C42 pad 1: +3V3 -> /MCU/RUN#
- C43 pad 1: +3V3 -> /MCU/STOP#
- C44 pad 1: +3V3 -> /MCU/KILL#
- C48 pad 1: +5V -> +3V3
- C49 pad 1: Net-(J11-VBUS) -> +3V3
- C50 pad 1: Net-(J11-VBUS) -> +3V3
- C51 pad 1: /VDD12DSI -> +3V3
- C52 pad 1: /VDD12DSI -> +3V3
- C53 pad 1: +3.3VA -> +3V3
- C54 pad 1: +3.3VA -> /MCU/VDD12DSI
- C55 pad 1: /RESET# -> /MCU/VDD12DSI
- C58 pad 1: Net-(U12-PH0) -> /Connectivity/RESET#
- C59 pad 1: Net-(U12-PH1) -> +3.3VA
- C6 pad 1: +3V3 -> Net-(U1-SS/TR)
- C60 pad 1: Net-(U12-VCAP1) -> +3.3VA
- C61 pad 1: Net-(U12-VCAP2) -> Net-(U14-PH0)
- C62 pad 1: Net-(U12-PC15) -> Net-(U14-PH1)
- C63 pad 1: Net-(U12-PC14) -> Net-(U14-VCAP1)
- C7 pad 1: +3V3 -> +12V
- C8 pad 1: Net-(U1-SS/TR) -> +3V3
- C9 pad 1: GND1 -> Net-(IC1-FB)
- C9 pad 2: Net-(IC1-VDD1) -> /Power/+12V_ISOLATED
- D3 pad 1: GND1 -> /Power/L_RECTIFIED
- D3 pad 3: Net-(D3-COM) -> NEUT
- D4 pad 1: /L_RECTIFIED -> GND
- D4 pad 2: GND1 -> Net-(D4-A)
- D5 pad 1: GND -> GND1
- D5 pad 2: Net-(D5-A) -> GND1
- D6 pad 1: Net-(D6-K) -> /MCU/RUN#
- D6 pad 2: +3V3 -> Net-(D6-A)
- D7 pad 1: Net-(D7-K) -> /MCU/STOP#
- D7 pad 2: +3V3 -> Net-(D7-A)
- D8 pad 1: Net-(D8-K) -> /MCU/KILL#
- D8 pad 2: +3V3 -> Net-(D8-A)
- H3 pad 1: Earth -> /SHIELD
- H4 pad 1: Earth -> /SHIELD
- HS1 pad 1: (no net) -> Earth
- HS2 pad 1: (no net) -> Earth
- HS3 pad 1: (no net) -> Earth
- HS4 pad 1: (no net) -> Earth
- IC1 pad 1: Net-(IC1-VDD1) -> Net-(IC1-PG)
- IC1 pad 2: Net-(IC1-INP) -> GND1
- IC1 pad 3: GND1 -> Net-(IC1-FB)
- IC1 pad 4: GND1 -> /Power/+12V_ISOLATED
- IC1 pad 5: GND -> Net-(IC1-VB)
- IC1 pad 6: unconnected-(IC1-OUT1-Pad6) -> Net-(IC1-VB)
- IC1 pad 7: /AC_SYNC -> unconnected-(IC1-NC-Pad7)
- IC1 pad 8: +3V3 -> /Power/L_RECTIFIED
- IC2 pad 1: Net-(IC2-PG) -> Net-(IC2-VDD1)
- IC2 pad 2: GND1 -> Net-(IC2-INP)
- IC2 pad 3: Net-(IC2-FB) -> GND1
- IC2 pad 4: /+12V_ISOLATED -> GND1
- IC2 pad 5: Net-(IC2-VB) -> GND
- IC2 pad 6: Net-(IC2-VB) -> unconnected-(IC2-OUT1-Pad6)
- IC2 pad 7: unconnected-(IC2-NC-Pad7) -> /AC Synchronization/AC_SYNC
- IC2 pad 8: /L_RECTIFIED -> +3V3
- J1 pad 1: /L_FUSED -> NEUT
- J1 pad 3: /N -> LINE
- J10 pad 1: /TC4+ -> Net-(J10-VBUS)
- J10 pad 2: /TC4- -> /Connectivity/USB_D-
- J13 pad 1: +3V3 -> GND
- J13 pad 10: /RESET# -> GND
- J13 pad 2: /SWDIO -> Net-(J13-Pad2)
- J13 pad 3: GND -> Net-(J13-Pad3)
- J13 pad 4: /SWCLK -> GND
- J13 pad 5: GND -> Net-(J13-Pad5)
- J13 pad 6: /SWO -> Net-(J13-Pad6)
- J13 pad 7: unconnected-(J13-KEY-Pad7) -> GND
- J13 pad 8: unconnected-(J13-NC/TDI-Pad8) -> Net-(J13-Pad8)
- J13 pad 9: Earth -> Net-(J13-Pad9)
- J2 pad 2: /N -> NEUT
- J3 pad 2: /N -> NEUT
- J4 pad 1: GND -> Net-(Q3-A1)
- J4 pad 2: Net-(J4-Pad2) -> NEUT
- J5 pad 1: Net-(Q3-A1) -> Net-(Q4-A1)
- J5 pad 2: /N -> NEUT
- J6 pad 1: Net-(Q4-A1) -> /Thermocouples/TC1+
- J6 pad 2: /N -> /Thermocouples/TC1-
- J7 pad 1: /TC1+ -> /Thermocouples/TC3+
- J7 pad 2: /TC1- -> /Thermocouples/TC3-
- J8 pad 1: /TC2+ -> /Thermocouples/TC2+
- J8 pad 2: /TC2- -> /Thermocouples/TC2-
- J9 pad 1: /TC3+ -> /Thermocouples/TC4+
- J9 pad 2: /TC3- -> /Thermocouples/TC4-
- L1 pad 1: +3V3 -> GND
- L1 pad 2: +3.3VA -> Earth
- L4 pad 1: GND -> +3V3
- L4 pad 2: Earth -> +3.3VA
- M1 pad 3: /FANS_OUT_TACHO -> /Fans/FANS_IN_TACHO
- M1 pad 4: /FANS_OUT_PWM -> /Fans/FANS_IN_PWM
- M2 pad 4: /FANS_OUT_PWM -> /Fans/FANS_IN_PWM
- M3 pad 3: /FANS_IN_TACHO -> /Fans/FANS_OUT_TACHO
- M3 pad 4: /FANS_IN_PWM -> /Fans/FANS_OUT_PWM
- M4 pad 4: /FANS_IN_PWM -> /Fans/FANS_OUT_PWM
- Q1 pad 2: /L_FUSED -> LINE
- Q2 pad 2: /L_FUSED -> LINE
- Q3 pad 2: /L_FUSED -> LINE
- Q4 pad 2: /L_FUSED -> LINE
- R10 pad 1: /DSI1_DP0 -> /Power/+12V_ISOLATED
- R10 pad 2: Net-(J4-Pad9) -> Net-(IC1-FB)
- R11 pad 1: Net-(R11-Pad1) -> GND1
- R11 pad 2: /L_FUSED -> Net-(IC1-FB)
- R12 pad 1: Net-(R12-Pad1) -> +3V3
- R12 pad 2: /L_FUSED -> Net-(U3-PG)
- R13 pad 1: /+12V_ISOLATED -> Net-(U3-FB)
- R13 pad 2: Net-(IC1-VDD1) -> GND
- R14 pad 1: /DSI1_DN1 -> /AC Synchronization/+12V_ISOLATED
- R14 pad 2: Net-(J4-Pad2) -> Net-(IC2-VDD1)
- R15 pad 1: /DSI1_DP1 -> LINE
- R15 pad 2: Net-(J4-Pad3) -> Net-(R15-Pad2)
- R16 pad 1: /LCD_SCL -> Net-(R15-Pad2)
- R16 pad 2: Net-(J4-Pad11) -> Net-(R16-Pad2)
- R17 pad 1: /LCD_SDA -> Net-(R16-Pad2)
- R17 pad 2: Net-(J4-Pad12) -> Net-(D5-COM)
- R18 pad 1: /L_FUSED -> Net-(D5-COM)
- R18 pad 2: Net-(C12-Pad1) -> Net-(IC2-INP)
- R19 pad 1: /L_FUSED -> +5V
- R19 pad 2: Net-(C13-Pad1) -> Net-(R19-Pad2)
- R20 pad 1: /L_FUSED -> +5V
- R21 pad 1: Net-(R20-Pad2) -> Net-(R21-Pad1)
- R21 pad 2: Net-(R21-Pad2) -> LINE
- R22 pad 1: Net-(R21-Pad2) -> Net-(R22-Pad1)
- R22 pad 2: Net-(D3-COM) -> LINE
- R23 pad 1: Net-(D3-COM) -> LINE
- R23 pad 2: Net-(IC1-INP) -> Net-(C19-Pad1)
- R24 pad 1: +5V -> LINE
- R24 pad 2: Net-(R24-Pad2) -> Net-(C20-Pad1)
- R26 pad 1: Net-(IC2-PG) -> +5V
- R26 pad 2: /+12V_ISOLATED -> Net-(R26-Pad2)
- R27 pad 1: +3V3 -> Net-(R27-Pad1)
- R27 pad 2: Net-(D5-A) -> LINE
- R28 pad 1: +3V3 -> Net-(R28-Pad1)
- R28 pad 2: Net-(U5-FB) -> LINE
- R29 pad 1: /+12V_ISOLATED -> LINE
- R29 pad 2: Net-(IC2-FB) -> Net-(C21-Pad1)
- R30 pad 1: GND1 -> LINE
- R30 pad 2: Net-(IC2-FB) -> Net-(C22-Pad1)
- R31 pad 1: +3V3 -> /Thermocouples/TC1+
- R31 pad 2: Net-(U5-PG) -> +5V
- R32 pad 1: Net-(U5-FB) -> GND
- R32 pad 2: GND -> /Thermocouples/TC1-
- R33 pad 1: Net-(R33-Pad1) -> /Thermocouples/TC3+
- R33 pad 2: /L_FUSED -> +5V
- R34 pad 1: Net-(R34-Pad1) -> GND
- R34 pad 2: /L_FUSED -> /Thermocouples/TC3-
- R35 pad 1: /L_FUSED -> /Thermocouples/TC1+
- R35 pad 2: Net-(C21-Pad1) -> Net-(U8-AIN0)
- R36 pad 1: /L_FUSED -> /Thermocouples/TC1-
- R36 pad 2: Net-(C22-Pad1) -> Net-(U8-AIN1)
- R37 pad 1: +5V -> /Thermocouples/TC3+
- R37 pad 2: Net-(R37-Pad2) -> Net-(U8-AIN2)
- R38 pad 1: +5V -> /Thermocouples/TC3-
- R38 pad 2: Net-(R38-Pad2) -> Net-(U8-AIN3)
- R39 pad 1: +3V3 -> /Thermocouples/TC2+
- R39 pad 2: /RUN# -> +5V
- R4 pad 1: /DSI1_CN -> NEUT
- R4 pad 2: Net-(J4-Pad5) -> Net-(C1-Pad1)
- R40 pad 1: +3V3 -> GND
- R40 pad 2: /STOP# -> /Thermocouples/TC2-
- R41 pad 1: +3V3 -> /Thermocouples/TC4+
- R41 pad 2: /KILL# -> +5V
- R42 pad 1: Net-(LS1--) -> GND
- R42 pad 2: +3V3 -> /Thermocouples/TC4-
- R43 pad 1: +3V3 -> /Thermocouples/TC2+
- R43 pad 2: /TRIAC_A_ON# -> Net-(U9-AIN0)
- R44 pad 1: +3V3 -> /Thermocouples/TC2-
- R44 pad 2: /USER_IN4# -> Net-(U9-AIN1)
- R45 pad 1: +3V3 -> /Thermocouples/TC4+
- R45 pad 2: /TRIAC_B_ON# -> Net-(U9-AIN2)
- R46 pad 1: +3V3 -> /Thermocouples/TC4-
- R46 pad 2: /USER_IN3# -> Net-(U9-AIN3)
- R47 pad 1: /DIODE_RUN# -> /Connectivity/USB_OC#
- R47 pad 2: Net-(D6-K) -> +5V
- R48 pad 1: /DIODE_STOP# -> /Connectivity/USB_EN#
- R48 pad 2: Net-(D7-K) -> +5V
- R49 pad 1: /DIODE_HEAT# -> GND
- R49 pad 2: Net-(D8-K) -> Net-(J11-CC2)
- R5 pad 1: /DSI1_CP -> +5V
- R5 pad 2: Net-(J4-Pad6) -> Net-(U1-PG)
- R50 pad 1: /DIODE_COOL# -> GND
- R50 pad 2: Net-(D9-K) -> Net-(J11-CC1)
- R51 pad 1: /DIODE_FAIL# -> Net-(J11-VBUS-PadA4)
- R51 pad 2: Net-(D10-K) -> /Connectivity/USB_UART_VBUS_SENSE
- R52 pad 1: /DIODE_TEST# -> /Connectivity/USB_UART_VBUS_SENSE
- R52 pad 2: Net-(D11-K) -> GND
- R53 pad 1: /BUZZER_ON -> +3V3
- R53 pad 2: Net-(Q5-B) -> Net-(D6-A)
- R54 pad 2: /TRIAC_C_ON# -> Net-(D7-A)
- R55 pad 2: /USER_IN2# -> Net-(D8-A)
- R56 pad 1: +3V3 -> /MCU/RUN#
- R56 pad 2: /TRIAC_D_ON# -> Net-(D6-A)
- R57 pad 1: +3V3 -> /MCU/STOP#
- R57 pad 2: /USER_IN1# -> Net-(D7-A)
- R58 pad 1: /TC1+ -> /MCU/KILL#
- R58 pad 2: +5V -> Net-(D8-A)
- R59 pad 1: /TC2+ -> Net-(LS1--)
- R59 pad 2: +5V -> +3V3
- R6 pad 1: /L_FUSED -> Net-(U1-FB)
- R6 pad 2: Net-(C1-Pad1) -> GND
- R60 pad 1: /TC1+ -> /MCU/DIODE_RUN#
- R60 pad 2: Net-(U8-AIN0) -> Net-(D9-K)
- R61 pad 1: /TC2+ -> /MCU/DIODE_STOP#
- R61 pad 2: Net-(U9-AIN0) -> Net-(D10-K)
- R62 pad 1: /TC1- -> /MCU/DIODE_HEAT#
- R62 pad 2: Net-(U8-AIN1) -> Net-(D11-K)
- R63 pad 1: /TC2- -> /MCU/DIODE_COOL#
- R63 pad 2: Net-(U9-AIN1) -> Net-(D12-K)
- R64 pad 1: GND -> /MCU/DIODE_FAIL#
- R64 pad 2: /TC1- -> Net-(D13-K)
- R65 pad 1: GND -> /MCU/DIODE_TEST#
- R65 pad 2: /TC2- -> Net-(D14-K)
- R66 pad 1: /TC3+ -> /MCU/BUZZER_ON
- R66 pad 2: +5V -> Net-(Q5-B)
- R67 pad 1: /TC4+ -> /MCU/DSI1_CN
- R67 pad 2: +5V -> Net-(J13-Pad5)
- R68 pad 1: /TC3+ -> /MCU/DSI1_CP
- R68 pad 2: Net-(U8-AIN2) -> Net-(J13-Pad6)
- R69 pad 1: /TC4+ -> /User Interface/LCD/DSI1_DN0
- R69 pad 2: Net-(U9-AIN2) -> Net-(J13-Pad8)
- R7 pad 1: +5V -> Net-(IC1-PG)
- R7 pad 2: Net-(U1-PG) -> /Power/+12V_ISOLATED
- R70 pad 1: /TC3- -> /User Interface/LCD/DSI1_DP0
- R70 pad 2: Net-(U8-AIN3) -> Net-(J13-Pad9)
- R71 pad 1: /TC4- -> /User Interface/LCD/DSI1_DN1
- R71 pad 2: Net-(U9-AIN3) -> Net-(J13-Pad2)
- R72 pad 1: GND -> /User Interface/LCD/DSI1_DP1
- R72 pad 2: /TC3- -> Net-(J13-Pad3)
- R73 pad 1: GND -> /User Interface/LCD/LCD_SCL
- R73 pad 2: /TC4- -> Net-(J13-Pad11)
- R74 pad 1: /USB_OC# -> /User Interface/LCD/LCD_SDA
- R74 pad 2: +5V -> Net-(J13-Pad12)
- R75 pad 2: /VDD12DSI -> /Device Configuration/TRIAC_A_ON#
- R76 pad 1: /USB_EN# -> +3V3
- R76 pad 2: +5V -> /Device Configuration/TRIAC_B_ON#
- R77 pad 1: Net-(SW7-C) -> +3V3
- R77 pad 2: Net-(U12-BOOT0) -> /Device Configuration/TRIAC_C_ON#
- R78 pad 1: Net-(U12-PB2) -> +3V3
- R78 pad 2: Net-(SW8-C) -> /Device Configuration/TRIAC_D_ON#
- R79 pad 1: GND -> +3V3
- R79 pad 2: Net-(J12-CC2) -> /Device Configuration/USER_IN4#
- R8 pad 1: Net-(U1-FB) -> +3V3
- R8 pad 2: GND -> Net-(D4-A)
- R80 pad 1: GND -> +3V3
- R80 pad 2: Net-(J12-CC1) -> /Device Configuration/USER_IN3#
- R81 pad 1: Net-(J12-VBUS-PadA4) -> +3V3
- R81 pad 2: /USB_UART_VBUS_SENSE -> /Device Configuration/USER_IN2#
- R82 pad 1: /USB_UART_VBUS_SENSE -> +3V3
- R82 pad 2: GND -> /Device Configuration/USER_IN1#
- R9 pad 1: /DSI1_DN0 -> +3V3
- R9 pad 2: Net-(J4-Pad8) -> Net-(U3-FB)
- RV1 pad 1: /L_FUSED -> LINE
- RV2 pad 1: /L_FUSED -> LINE
- RV3 pad 1: /L_FUSED -> LINE
- RV4 pad 1: /L_FUSED -> LINE
- SW2 pad 1: /TRIAC_A_ON# -> Net-(D6-A)
- SW2 pad 2: /TRIAC_B_ON# -> GND
- SW3 pad 1: /RUN# -> Net-(D7-A)
- SW4 pad 1: /STOP# -> Net-(D8-A)
- SW5 pad 1: /KILL# -> /Device Configuration/TRIAC_A_ON#
- SW5 pad 2: GND -> /Device Configuration/TRIAC_B_ON#
- SW6 pad 2: /RESET# -> /Connectivity/RESET#
- TP1 pad 1: /DSI1_CN -> +5V
- TP10 pad 1: /LCD_SDA -> /Heaters/HEATER_C#
- TP11 pad 1: /AC_SYNC -> /Heaters/HEATER_B#
- TP12 pad 1: Net-(IC1-INP) -> /Heaters/HEATER_D#
- TP13 pad 1: /HEATER_A# -> /Heaters/HEATER_B#
- TP14 pad 1: /HEATER_B# -> /Heaters/HEATER_D#
- TP15 pad 1: /HEATER_A# -> Net-(U8-AIN2)
- TP16 pad 1: /HEATER_B# -> Net-(U8-AIN0)
- TP17 pad 1: +3V3 -> /MCU/SPI_TC1_MISO
- TP18 pad 1: /+12V_ISOLATED -> /MCU/SPI_TC1_CLK
- TP19 pad 1: /HEATER_C# -> /MCU/SPI_TC1_MOSI
- TP2 pad 1: /DSI1_CP -> +12V
- TP20 pad 1: /HEATER_D# -> Net-(U9-AIN2)
- TP21 pad 1: /HEATER_C# -> Net-(U9-AIN0)
- TP22 pad 1: /HEATER_D# -> /Thermocouples/SPI_TC2_MISO
- TP23 pad 1: Net-(U8-AIN0) -> /Thermocouples/SPI_TC2_CLK
- TP24 pad 1: Net-(U9-AIN0) -> /Thermocouples/SPI_TC2_MOSI
- TP25 pad 1: /SPI_TC1_CLK -> Net-(J10-VBUS)
- TP26 pad 1: /SPI_TC2_CLK -> /Connectivity/RESET#
- TP27 pad 1: /SPI_TC1_MOSI -> /Connectivity/SWCLK
- TP28 pad 1: /SPI_TC2_MOSI -> /Connectivity/SWDIO
- TP29 pad 1: /SPI_TC1_MISO -> /Connectivity/SWO
- TP3 pad 1: /DSI1_DN0 -> +3V3
- TP30 pad 1: /SPI_TC2_MISO -> /MCU/DSI1_CP
- TP31 pad 1: Net-(U8-AIN2) -> /User Interface/LCD/DSI1_DN0
- TP32 pad 1: Net-(U9-AIN2) -> /MCU/DSI1_CN
- TP33 pad 1: Net-(J11-VBUS) -> /User Interface/LCD/DSI1_DP0
- TP34 pad 1: +3.3VA -> /User Interface/LCD/DSI1_DP1
- TP35 pad 1: Net-(U12-PH0) -> /User Interface/LCD/LCD_SCL
- TP36 pad 1: Net-(U12-PC14) -> /User Interface/LCD/DSI1_DN1
- TP37 pad 1: /RESET# -> /User Interface/LCD/LCD_SDA
- TP38 pad 1: /SWCLK -> +3.3VA
- TP39 pad 1: /SWDIO -> Net-(U14-PH0)
- TP4 pad 1: +5V -> /Power/+12V_ISOLATED
- TP40 pad 1: /SWO -> Net-(U14-PC14)
- TP5 pad 1: +12V -> /AC Synchronization/AC_SYNC
- TP6 pad 1: /DSI1_DP0 -> Net-(IC2-INP)
- TP7 pad 1: /DSI1_DN1 -> /Heaters/HEATER_A#
- TP8 pad 1: /DSI1_DP1 -> /Heaters/HEATER_C#
- TP9 pad 1: /LCD_SCL -> /Heaters/HEATER_A#
- U10 pad 1: Net-(J11-VBUS) -> Net-(J10-VBUS)
- U10 pad 3: /USB_OC# -> /Connectivity/USB_OC#
- U10 pad 4: /USB_EN# -> /Connectivity/USB_EN#
- U11 pad 1: /USB_D- -> /Connectivity/USB_D-
- U11 pad 5: Net-(J11-VBUS) -> Net-(J10-VBUS)
- U11 pad 6: /USB_D+ -> /Connectivity/USB_D+
- U12 pad 1: unconnected-(U12-PE2-Pad1) -> /Connectivity/USB_UART_D-
- U12 pad 2: GND -> Earth
- U12 pad 3: +3V3 -> unconnected-(U12-Pad3)
- U12 pad 5: Net-(U12-PC14) -> Net-(J11-VBUS-PadA4)
- U12 pad 6: Net-(U12-PC15) -> /Connectivity/USB_UART_D+
- U13 pad 1: /USB_UART_D- -> /Connectivity/SWDIO
- U13 pad 4: unconnected-(U13-Pad4) -> /Connectivity/SWO
- U13 pad 5: Net-(J12-VBUS-PadA4) -> +3V3
- U13 pad 6: /USB_UART_D+ -> /Connectivity/SWCLK
- U14 pad 1: /SWDIO -> unconnected-(U14-PE2-Pad1)
- U14 pad 2: Earth -> GND
- U14 pad 3: unconnected-(U14-Pad3) -> +3V3
- U14 pad 4: /SWO -> unconnected-(U14-PC13-Pad4)
- U14 pad 5: +3V3 -> Net-(U14-PC14)
- U14 pad 6: /SWCLK -> Net-(U14-PC15)
- U2 pad 1: /L_FUSED -> NEUT
- U2 pad 2: /N -> LINE
- U3 pad 1: Net-(R24-Pad2) -> +12V
- U3 pad 2: /HEATER_A# -> +12V
- U3 pad 3: unconnected-(U3-NC-Pad3) -> GND
- U3 pad 4: Net-(Q1-G) -> +3V3
- U3 pad 5: unconnected-(U3-NC-Pad5) -> +3V3
- U3 pad 6: Net-(R11-Pad1) -> Net-(U3-FB)
- U4 pad 1: Net-(R25-Pad2) -> Net-(R19-Pad2)
- U4 pad 2: /HEATER_B# -> /Heaters/HEATER_A#
- U4 pad 4: Net-(Q2-G) -> Net-(Q1-G)
- U4 pad 6: Net-(R12-Pad1) -> Net-(R21-Pad1)
- U5 pad 1: +12V -> Net-(R20-Pad2)
- U5 pad 2: +12V -> /Heaters/HEATER_C#
- U5 pad 3: GND -> unconnected-(U5-NC-Pad3)
- U5 pad 4: +3V3 -> Net-(Q2-G)
- U5 pad 5: +3V3 -> unconnected-(U5-NC-Pad5)
- U5 pad 6: Net-(U5-FB) -> Net-(R22-Pad1)
- U6 pad 1: Net-(R37-Pad2) -> Net-(R25-Pad2)
- U6 pad 2: /HEATER_C# -> /Heaters/HEATER_B#
- U6 pad 6: Net-(R33-Pad1) -> Net-(R27-Pad1)
- U7 pad 1: Net-(R38-Pad2) -> Net-(R26-Pad2)
- U7 pad 2: /HEATER_D# -> /Heaters/HEATER_D#
- U7 pad 6: Net-(R34-Pad1) -> Net-(R28-Pad1)
- U8 pad 1: /SPI_TC1_CLK -> /MCU/SPI_TC1_CLK
- U8 pad 10: /SPI_TC1_MOSI -> /MCU/SPI_TC1_MOSI
- U8 pad 9: /SPI_TC1_MISO -> /MCU/SPI_TC1_MISO
- U9 pad 1: /SPI_TC2_CLK -> /Thermocouples/SPI_TC2_CLK
- U9 pad 10: /SPI_TC2_MOSI -> /Thermocouples/SPI_TC2_MOSI
- U9 pad 9: /SPI_TC2_MISO -> /Thermocouples/SPI_TC2_MISO
- Y1 pad 1: Net-(U12-PH1) -> Net-(U14-PH1)
- Y1 pad 3: Net-(U12-PH0) -> Net-(U14-PH0)
- Y2 pad 1: Net-(U12-PC15) -> Net-(U14-PC15)
- Y2 pad 2: Net-(U12-PC14) -> Net-(U14-PC14)
Routing:
- net LINE: track 0.00 -> 345.7 mm, vias 0 -> 2
- net /L_FUSED: track 317.4 -> 0.00 mm
- net NEUT: track 0.00 -> 216.6 mm
- net /N: track 210.6 -> 0.00 mm
- net Net-(Q3-G): track 23.7 -> 7.11 mm, vias 1 -> 0
- net Net-(C1-Pad1): track 23.1 -> 7.80 mm, vias 1 -> 0
- net Net-(D3-COM): track 14.3 -> 0.00 mm
- net /L_RECTIFIED: track 14.0 -> 0.00 mm
- net Net-(R28-Pad1): track 0.00 -> 12.5 mm
- net Net-(C12-Pad1): track 9.18 -> 0.00 mm
- net Net-(C13-Pad1): track 9.17 -> 0.00 mm
- net GND1: track 8.15 -> 0.00 mm
- net Net-(Q2-A1): track 43.9 -> 51.4 mm
- net Net-(R22-Pad1): track 0.00 -> 6.79 mm
- net Net-(R27-Pad1): track 0.00 -> 6.67 mm
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Other:
- board size 170 x 100 mm -> 180 x 110 mm
