File: config.kicad_sch (KiCad schematic)
At the start: 9 parts, among them SW5 SW_DIP_x08

Commit message: feat: add board dimensions and change mcu position
Parts:
- renumbered R79 to R76, R76 to R77, R80 to R78, R77 to R79, R81 to R80, R78 to R81
Changed lines of the file:
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@@
 		(dnp no)
 		(fields_autoplaced yes)
-		(property "Reference" "R81"
+		(property "Reference" "R80"
 			(at 158.75 111.76 90)
 			(show_name no)
@@
 			(project "reflow_station"
 				(path "/77770e37-dda2-4cf3-b2f1-cea4793bc3be/e571f478-2f31-4f14-9227-de33168fc084"
-					(reference "R81")
+					(reference "R80")
 					(unit 1)
 				)
@@
 		(dnp no)
 		(fields_autoplaced yes)
-		(property "Reference" "R76"
+		(property "Reference" "R77"
 			(at 120.65 101.6 90)
 			(show_name no)
@@
 			(project "reflow_station"
 				(path "/77770e37-dda2-4cf3-b2f1-cea4793bc3be/e571f478-2f31-4f14-9227-de33168fc084"
-					(reference "R76")
+					(reference "R77")
 					(unit 1)
 				)
@@
 		(dnp no)
 		(fields_autoplaced yes)
-		(property "Reference" "R77"
+		(property "Reference" "R79"
 			(at 120.65 111.76 90)
 			(show_name no)
@@
 			(project "reflow_station"
 				(path "/77770e37-dda2-4cf3-b2f1-cea4793bc3be/e571f478-2f31-4f14-9227-de33168fc084"
-					(reference "R77")
+					(reference "R79")
 					(unit 1)
 				)
@@
 		(dnp no)
 		(fields_autoplaced yes)
-		(property "Reference" "#PWR0136"
+		(property "Reference" "#PWR0139"
 			(at 130.81 66.04 0)
 			(hide yes)
@@
 			(project "reflow_station"
 				(path "/77770e37-dda2-4cf3-b2f1-cea4793bc3be/e571f478-2f31-4f14-9227-de33168fc084"
-					(reference "#PWR0136")
+					(reference "#PWR0139")
 					(unit 1)
 				)
@@
 		(dnp no)
 		(fields_autoplaced yes)
-		(property "Reference" "#PWR0135"
+		(property "Reference" "#PWR0140"
 			(at 114.3 97.79 0)
 			(hide yes)
@@
 			(project "reflow_station"
 				(path "/77770e37-dda2-4cf3-b2f1-cea4793bc3be/e571f478-2f31-4f14-9227-de33168fc084"
-					(reference "#PWR0135")
+					(reference "#PWR0140")
 					(unit 1)
 				)
@@
 		(dnp no)
 		(fields_autoplaced yes)
-		(property "Reference" "R78"
+		(property "Reference" "R81"
 			(at 120.65 120.65 90)
 			(show_name no)
@@
 			(project "reflow_station"
 				(path "/77770e37-dda2-4cf3-b2f1-cea4793bc3be/e571f478-2f31-4f14-9227-de33168fc084"
-					(reference "R78")
+					(reference "R81")
 					(unit 1)
 				)
@@
 		(in_pos_files yes)
 		(dnp no)
-		(property "Reference" "#PWR0137"
+		(property "Reference" "#PWR0141"
 			(at 165.1 97.79 0)
 			(hide yes)
@@
 			(project "reflow_station"
 				(path "/77770e37-dda2-4cf3-b2f1-cea4793bc3be/e571f478-2f31-4f14-9227-de33168fc084"
-					(reference "#PWR0137")
+					(reference "#PWR0141")
 					(unit 1)
 				)
@@
 		(dnp no)
 		(fields_autoplaced yes)
-		(property "Reference" "R79"
+		(property "Reference" "R76"
 			(at 158.75 92.71 90)
 			(show_name no)
@@
 			(project "reflow_station"
 				(path "/77770e37-dda2-4cf3-b2f1-cea4793bc3be/e571f478-2f31-4f14-9227-de33168fc084"
-					(reference "R79")
+					(reference "R76")
 					(unit 1)
 				)
@@
 		(dnp no)
 		(fields_autoplaced yes)
-		(property "Reference" "R80"
+		(property "Reference" "R78"
 			(at 158.75 101.6 90)
 			(show_name no)
@@
 			(project "reflow_station"
 				(path "/77770e37-dda2-4cf3-b2f1-cea4793bc3be/e571f478-2f31-4f14-9227-de33168fc084"
-					(reference "R80")
+					(reference "R78")
 					(unit 1)
 				)

Commit message: feat: add ground and earth(shield) planes, add better - multi layer connection for AC mains connector
Parts:
- renumbered R77 to R76, R79 to R77, R81 to R78, R76 to R79, R78 to R80, R80 to R81
Changed lines of the file:
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@@
 		(dnp no)
 		(fields_autoplaced yes)
-		(property "Reference" "R80"
+		(property "Reference" "R81"
 			(at 158.75 111.76 90)
 			(show_name no)
@@
 			(project "reflow_station"
 				(path "/77770e37-dda2-4cf3-b2f1-cea4793bc3be/e571f478-2f31-4f14-9227-de33168fc084"
-					(reference "R80")
+					(reference "R81")
 					(unit 1)
 				)
@@
 		(dnp no)
 		(fields_autoplaced yes)
-		(property "Reference" "R77"
+		(property "Reference" "R76"
 			(at 120.65 101.6 90)
 			(show_name no)
@@
 			(project "reflow_station"
 				(path "/77770e37-dda2-4cf3-b2f1-cea4793bc3be/e571f478-2f31-4f14-9227-de33168fc084"
-					(reference "R77")
+					(reference "R76")
 					(unit 1)
 				)
@@
 		(dnp no)
 		(fields_autoplaced yes)
-		(property "Reference" "R79"
+		(property "Reference" "R77"
 			(at 120.65 111.76 90)
 			(show_name no)
@@
 			(project "reflow_station"
 				(path "/77770e37-dda2-4cf3-b2f1-cea4793bc3be/e571f478-2f31-4f14-9227-de33168fc084"
-					(reference "R79")
+					(reference "R77")
 					(unit 1)
 				)
@@
 		(dnp no)
 		(fields_autoplaced yes)
-		(property "Reference" "#PWR0139"
+		(property "Reference" "#PWR0140"
 			(at 130.81 66.04 0)
 			(hide yes)
@@
 			(project "reflow_station"
 				(path "/77770e37-dda2-4cf3-b2f1-cea4793bc3be/e571f478-2f31-4f14-9227-de33168fc084"
-					(reference "#PWR0139")
+					(reference "#PWR0140")
 					(unit 1)
 				)
@@
 		(dnp no)
 		(fields_autoplaced yes)
-		(property "Reference" "#PWR0140"
+		(property "Reference" "#PWR0139"
 			(at 114.3 97.79 0)
 			(hide yes)
@@
 			(project "reflow_station"
 				(path "/77770e37-dda2-4cf3-b2f1-cea4793bc3be/e571f478-2f31-4f14-9227-de33168fc084"
-					(reference "#PWR0140")
+					(reference "#PWR0139")
 					(unit 1)
 				)
@@
 		(dnp no)
 		(fields_autoplaced yes)
-		(property "Reference" "R81"
+		(property "Reference" "R78"
 			(at 120.65 120.65 90)
 			(show_name no)
@@
 			(project "reflow_station"
 				(path "/77770e37-dda2-4cf3-b2f1-cea4793bc3be/e571f478-2f31-4f14-9227-de33168fc084"
-					(reference "R81")
+					(reference "R78")
 					(unit 1)
 				)
@@
 		(dnp no)
 		(fields_autoplaced yes)
-		(property "Reference" "R76"
+		(property "Reference" "R79"
 			(at 158.75 92.71 90)
 			(show_name no)
@@
 			(project "reflow_station"
 				(path "/77770e37-dda2-4cf3-b2f1-cea4793bc3be/e571f478-2f31-4f14-9227-de33168fc084"
-					(reference "R76")
+					(reference "R79")
 					(unit 1)
 				)
@@
 		(dnp no)
 		(fields_autoplaced yes)
-		(property "Reference" "R78"
+		(property "Reference" "R80"
 			(at 158.75 101.6 90)
 			(show_name no)
@@
 			(project "reflow_station"
 				(path "/77770e37-dda2-4cf3-b2f1-cea4793bc3be/e571f478-2f31-4f14-9227-de33168fc084"
-					(reference "R78")
+					(reference "R80")
 					(unit 1)
 				)

Commit message: feat: route remaining traces
Parts:
- renumbered R75 to R81, R76 to R82, R77 to R83, R78 to R84, R79 to R85, R80 to R86, R81 to R87, R82 to R88
Changed lines of the file:
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@@
 		(dnp no)
 		(fields_autoplaced yes)
-		(property "Reference" "R81"
+		(property "Reference" "R87"
 			(at 158.75 111.76 90)
 			(show_name no)
@@
 			(project "reflow_station"
 				(path "/77770e37-dda2-4cf3-b2f1-cea4793bc3be/e571f478-2f31-4f14-9227-de33168fc084"
-					(reference "R81")
+					(reference "R87")
 					(unit 1)
 				)
@@
 		(dnp no)
 		(fields_autoplaced yes)
-		(property "Reference" "R76"
+		(property "Reference" "R82"
 			(at 120.65 101.6 90)
 			(show_name no)
@@
 			(project "reflow_station"
 				(path "/77770e37-dda2-4cf3-b2f1-cea4793bc3be/e571f478-2f31-4f14-9227-de33168fc084"
-					(reference "R76")
+					(reference "R82")
 					(unit 1)
 				)
@@
 		(dnp no)
 		(fields_autoplaced yes)
-		(property "Reference" "R77"
+		(property "Reference" "R83"
 			(at 120.65 111.76 90)
 			(show_name no)
@@
 			(project "reflow_station"
 				(path "/77770e37-dda2-4cf3-b2f1-cea4793bc3be/e571f478-2f31-4f14-9227-de33168fc084"
-					(reference "R77")
+					(reference "R83")
 					(unit 1)
 				)
@@
 		(dnp no)
 		(fields_autoplaced yes)
-		(property "Reference" "#PWR0140"
+		(property "Reference" "#PWR0141"
 			(at 130.81 66.04 0)
 			(hide yes)
@@
 			(project "reflow_station"
 				(path "/77770e37-dda2-4cf3-b2f1-cea4793bc3be/e571f478-2f31-4f14-9227-de33168fc084"
-					(reference "#PWR0140")
+					(reference "#PWR0141")
 					(unit 1)
 				)
@@
 		(dnp no)
 		(fields_autoplaced yes)
-		(property "Reference" "R75"
+		(property "Reference" "R81"
 			(at 120.65 92.71 90)
 			(show_name no)
@@
 			(project "reflow_station"
 				(path "/77770e37-dda2-4cf3-b2f1-cea4793bc3be/e571f478-2f31-4f14-9227-de33168fc084"
-					(reference "R75")
+					(reference "R81")
 					(unit 1)
 				)
@@
 		(dnp no)
 		(fields_autoplaced yes)
-		(property "Reference" "#PWR0139"
+		(property "Reference" "#PWR0140"
 			(at 114.3 97.79 0)
 			(hide yes)
@@
 			(project "reflow_station"
 				(path "/77770e37-dda2-4cf3-b2f1-cea4793bc3be/e571f478-2f31-4f14-9227-de33168fc084"
-					(reference "#PWR0139")
+					(reference "#PWR0140")
 					(unit 1)
 				)
@@
 		(dnp no)
 		(fields_autoplaced yes)
-		(property "Reference" "R78"
+		(property "Reference" "R84"
 			(at 120.65 120.65 90)
 			(show_name no)
@@
 			(project "reflow_station"
 				(path "/77770e37-dda2-4cf3-b2f1-cea4793bc3be/e571f478-2f31-4f14-9227-de33168fc084"
-					(reference "R78")
+					(reference "R84")
 					(unit 1)
 				)
@@
 		(in_pos_files yes)
 		(dnp no)
-		(property "Reference" "#PWR0141"
+		(property "Reference" "#PWR0142"
 			(at 165.1 97.79 0)
 			(hide yes)
@@
 			(project "reflow_station"
 				(path "/77770e37-dda2-4cf3-b2f1-cea4793bc3be/e571f478-2f31-4f14-9227-de33168fc084"
-					(reference "#PWR0141")
+					(reference "#PWR0142")
 					(unit 1)
 				)
@@
 		(dnp no)
 		(fields_autoplaced yes)
-		(property "Reference" "R79"
+		(property "Reference" "R85"
 			(at 158.75 92.71 90)
 			(show_name no)
@@
 			(project "reflow_station"
 				(path "/77770e37-dda2-4cf3-b2f1-cea4793bc3be/e571f478-2f31-4f14-9227-de33168fc084"
-					(reference "R79")
+					(reference "R85")
 					(unit 1)
 				)
@@
 		(dnp no)
 		(fields_autoplaced yes)
-		(property "Reference" "R80"
+		(property "Reference" "R86"
 			(at 158.75 101.6 90)
 			(show_name no)
@@
 			(project "reflow_station"
 				(path "/77770e37-dda2-4cf3-b2f1-cea4793bc3be/e571f478-2f31-4f14-9227-de33168fc084"
-					(reference "R80")
+					(reference "R86")
 					(unit 1)
 				)
@@
 		(dnp no)
 		(fields_autoplaced yes)
-		(property "Reference" "R82"
+		(property "Reference" "R88"
 			(at 158.75 120.65 90)
 			(show_name no)
@@
 			(project "reflow_station"
 				(path "/77770e37-dda2-4cf3-b2f1-cea4793bc3be/e571f478-2f31-4f14-9227-de33168fc084"
-					(reference "R82")
+					(reference "R88")
 					(unit 1)
 				)
