File: heaters.kicad_sch (KiCad schematic)
At the start: 44 parts, among them J2 1707027, J3 1707027, J4 1707027, J5 1707027, Q1 BTA16-600B, Q2 BTA16-600B, Q3 BTA16-600B, Q4 BTA16-600B, U4 MOC3052, U5 MOC3052, U6 MOC3052, U7 MOC3052

Commit message: feat: add board dimensions and change mcu position
Parts:
- removed TP10, TP13, TP14, TP9: TestPoint, reflow_station_library:TestPoint_Pad_D1.0mm, symbol reflow_station_symbols:TestPoint
- renumbered TP12 to TP10, TP11 to TP9

Commit message: feat: add power planes and move voltage regulators closer to their usage
Parts:
- R19, R20, R25, R26: value 680 -> 220; JLCPCB_PartNo C25130 -> C25091; Mfr.No 0402WGF6800TCE -> 0402WGF2200TCE; Supplier_Link https://jlcpcb.com/partdetail/25873-0402WGF6800TCE/C25130 -> https://jlcpcb.com/partdetail/25834-0402WGF2200TCE/C25091
Connections:
- net +5V renamed +3V3
