File: mcu.kicad_sch (KiCad schematic)
At the start: 35 parts, among them SW6 SW_Push, SW7 SW_SPDT, SW8 SW_SPDT, U14 STM32F469VIT6, Y1 25MHz, Y2 32.768kHz

Commit message: feat: add board dimensions and change mcu position
Parts:
- renumbered L4 to L6, TP38 to TP34, TP39 to TP35, TP40 to TP36

Commit message: feat: route thermocouples, USB ports and DSI
Parts:
- C55, C63, C64: footprint reflow_station_library:C_0603_1608Metric -> reflow_station_library:C_0402_1005Metric; JLCPCB_PartNo C23630 -> C12530; Mfr.No CL10A225KO8NNNC -> CL05A225MQ5NSNC; Package 0603 -> 0402; Supplier_Link https://jlcpcb.com/partdetail/24366-CL10A225KO8NNNC/C23630 -> https://jlcpcb.com/partdetail/13164-CL05A225MQ5NSNC/C12530
Changed lines of the file:
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@@
 			)
 		)
-		(property "Footprint" "reflow_station_library:C_0603_1608Metric"
+		(property "Footprint" "reflow_station_library:C_0402_1005Metric"
 			(at 127.9652 245.11 0)
 			(hide yes)
@@
 			)
 		)
-		(property "Description" "Unpolarized capacitor: 2.2uF 16V X5R 10% ceramic"
+		(property "Description" "Unpolarized capacitor: 2.2uF 6.3V X5R 20% ceramic"
 			(at 127 241.3 0)
 			(hide yes)
@@
 			)
 		)
-		(property "Supplier_Link" "https://jlcpcb.com/partdetail/24366-CL10A225KO8NNNC/C23630"
+		(property "Supplier_Link" "https://jlcpcb.com/partdetail/13164-CL05A225MQ5NSNC/C12530"
 			(at 127 241.3 0)
 			(hide yes)
@@
 			)
 		)
-		(property "JLCPCB_PartNo" "C23630"
+		(property "JLCPCB_PartNo" "C12530"
 			(at 127 241.3 0)
 			(hide yes)
@@
 			)
 		)
-		(property "Mfr.No" "CL10A225KO8NNNC"
+		(property "Mfr.No" "CL05A225MQ5NSNC"
 			(at 127 241.3 0)
 			(hide yes)
@@
 			)
 		)
-		(property "Package" "0603"
+		(property "Package" "0402"
 			(at 127 241.3 0)
 			(hide yes)
@@
 			)
 		)
-		(property "Footprint" "reflow_station_library:C_0603_1608Metric"
+		(property "Footprint" "reflow_station_library:C_0402_1005Metric"
 			(at 140.6652 245.11 0)
 			(hide yes)
@@
 			)
 		)
-		(property "Description" "Unpolarized capacitor: 2.2uF 16V X5R 10% ceramic"
+		(property "Description" "Unpolarized capacitor: 2.2uF 6.3V X5R 20% ceramic"
 			(at 139.7 241.3 0)
 			(hide yes)
@@
 			)
 		)
-		(property "Supplier_Link" "https://jlcpcb.com/partdetail/24366-CL10A225KO8NNNC/C23630"
+		(property "Supplier_Link" "https://jlcpcb.com/partdetail/13164-CL05A225MQ5NSNC/C12530"
 			(at 139.7 241.3 0)
 			(hide yes)
@@
 			)
 		)
-		(property "JLCPCB_PartNo" "C23630"
+		(property "JLCPCB_PartNo" "C12530"
 			(at 139.7 241.3 0)
 			(hide yes)
@@
 			)
 		)
-		(property "Mfr.No" "CL10A225KO8NNNC"
+		(property "Mfr.No" "CL05A225MQ5NSNC"
 			(at 139.7 241.3 0)
 			(hide yes)
@@
 			)
 		)
-		(property "Package" "0603"
+		(property "Package" "0402"
 			(at 139.7 241.3 0)
 			(hide yes)
@@
 			)
 		)
-		(property "Footprint" "reflow_station_library:C_0603_1608Metric"
+		(property "Footprint" "reflow_station_library:C_0402_1005Metric"
 			(at 173.6852 102.87 0)
 			(hide yes)
@@
 			)
 		)
-		(property "Description" "Unpolarized capacitor: 2.2uF 16V X5R 10% ceramic"
+		(property "Description" "Unpolarized capacitor: 2.2uF 6.3V X5R 20% ceramic"
 			(at 172.72 99.06 0)
 			(hide yes)
@@
 			)
 		)
-		(property "Supplier_Link" "https://jlcpcb.com/partdetail/24366-CL10A225KO8NNNC/C23630"
+		(property "Supplier_Link" "https://jlcpcb.com/partdetail/13164-CL05A225MQ5NSNC/C12530"
 			(at 172.72 99.06 0)
 			(hide yes)
@@
 			)
 		)
-		(property "JLCPCB_PartNo" "C23630"
+		(property "JLCPCB_PartNo" "C12530"
 			(at 172.72 99.06 0)
 			(hide yes)
@@
 			)
 		)
-		(property "Mfr.No" "CL10A225KO8NNNC"
+		(property "Mfr.No" "CL05A225MQ5NSNC"
 			(at 172.72 99.06 0)
 			(hide yes)
@@
 			)
 		)
-		(property "Package" "0603"
+		(property "Package" "0402"
 			(at 172.72 99.06 0)
 			(hide yes)

Commit message: feat: route config switches and SWD debug
Connections:
- net BOOT1: now also R85.2; no longer R85.1
- net at SW8.3 (C): now also R85.1; no longer R85.2
Other:
- moved on the sheet: R85
Changed lines of the file:
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@@
 	(symbol
 		(lib_id "reflow_station_symbols:R")
-		(at 267.97 172.72 90)
+		(at 267.97 172.72 270)
+		(mirror x)
 		(unit 1)
 		(body_style 1)
@@
 		(in_pos_files yes)
 		(dnp no)
-		(fields_autoplaced yes)
 		(property "Reference" "R85"
 			(at 267.97 166.37 90)

Commit message: feat: route remaining traces
Parts:
- renumbered R83 to R89, R84 to R90, R85 to R91, TP34 to TP28, TP35 to TP29, TP36 to TP30
