File: signaling.kicad_sch (KiCad schematic)
At the start: 16 parts, among them Q5 KSC1815YTA

Commit message: feat: route remaining traces
Parts:
- renumbered R59 to R65, R60 to R66, R61 to R67, R62 to R68, R63 to R69, R64 to R70, R65 to R71, R66 to R72
Changed lines of the file:
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@@
 		(in_pos_files yes)
 		(dnp no)
-		(property "Reference" "#PWR0127"
+		(property "Reference" "#PWR0128"
 			(at 182.88 86.36 0)
 			(hide yes)
@@
 			(project "reflow_station"
 				(path "/77770e37-dda2-4cf3-b2f1-cea4793bc3be/68b7f722-bad3-45c2-b522-78eb1b3727cc/3afc4fe4-3fa4-4c3e-afce-f70380747f42"
-					(reference "#PWR0127")
+					(reference "#PWR0128")
 					(unit 1)
 				)
@@
 		(in_pos_files yes)
 		(dnp no)
-		(property "Reference" "#PWR0121"
+		(property "Reference" "#PWR0122"
 			(at 243.84 82.55 0)
 			(hide yes)
@@
 			(project "reflow_station"
 				(path "/77770e37-dda2-4cf3-b2f1-cea4793bc3be/68b7f722-bad3-45c2-b522-78eb1b3727cc/3afc4fe4-3fa4-4c3e-afce-f70380747f42"
-					(reference "#PWR0121")
+					(reference "#PWR0122")
 					(unit 1)
 				)
@@
 		(dnp no)
 		(fields_autoplaced yes)
-		(property "Reference" "R65"
+		(property "Reference" "R71"
 			(at 185.42 100.3299 0)
 			(show_name no)
@@
 			(project "reflow_station"
 				(path "/77770e37-dda2-4cf3-b2f1-cea4793bc3be/68b7f722-bad3-45c2-b522-78eb1b3727cc/3afc4fe4-3fa4-4c3e-afce-f70380747f42"
-					(reference "R65")
+					(reference "R71")
 					(unit 1)
 				)
@@
 		(dnp no)
 		(fields_autoplaced yes)
-		(property "Reference" "#PWR0128"
+		(property "Reference" "#PWR0129"
 			(at 243.84 118.11 0)
 			(hide yes)
@@
 			(project "reflow_station"
 				(path "/77770e37-dda2-4cf3-b2f1-cea4793bc3be/68b7f722-bad3-45c2-b522-78eb1b3727cc/3afc4fe4-3fa4-4c3e-afce-f70380747f42"
-					(reference "#PWR0128")
+					(reference "#PWR0129")
 					(unit 1)
 				)
@@
 		(dnp no)
 		(fields_autoplaced yes)
-		(property "Reference" "R62"
+		(property "Reference" "R68"
 			(at 109.22 100.3299 0)
 			(show_name no)
@@
 			(project "reflow_station"
 				(path "/77770e37-dda2-4cf3-b2f1-cea4793bc3be/68b7f722-bad3-45c2-b522-78eb1b3727cc/3afc4fe4-3fa4-4c3e-afce-f70380747f42"
-					(reference "R62")
+					(reference "R68")
 					(unit 1)
 				)
@@
 		(in_pos_files yes)
 		(dnp no)
-		(property "Reference" "#PWR0125"
+		(property "Reference" "#PWR0126"
 			(at 132.08 86.36 0)
 			(hide yes)
@@
 			(project "reflow_station"
 				(path "/77770e37-dda2-4cf3-b2f1-cea4793bc3be/68b7f722-bad3-45c2-b522-78eb1b3727cc/3afc4fe4-3fa4-4c3e-afce-f70380747f42"
-					(reference "#PWR0125")
+					(reference "#PWR0126")
 					(unit 1)
 				)
@@
 		(dnp no)
 		(fields_autoplaced yes)
-		(property "Reference" "R61"
+		(property "Reference" "R67"
 			(at 83.82 100.3299 0)
 			(show_name no)
@@
 			(project "reflow_station"
 				(path "/77770e37-dda2-4cf3-b2f1-cea4793bc3be/68b7f722-bad3-45c2-b522-78eb1b3727cc/3afc4fe4-3fa4-4c3e-afce-f70380747f42"
-					(reference "R61")
+					(reference "R67")
 					(unit 1)
 				)
@@
 		(dnp no)
 		(fields_autoplaced yes)
-		(property "Reference" "R66"
+		(property "Reference" "R72"
 			(at 224.79 96.52 90)
 			(show_name no)
@@
 			(project "reflow_station"
 				(path "/77770e37-dda2-4cf3-b2f1-cea4793bc3be/68b7f722-bad3-45c2-b522-78eb1b3727cc/3afc4fe4-3fa4-4c3e-afce-f70380747f42"
-					(reference "R66")
+					(reference "R72")
 					(unit 1)
 				)
@@
 		(in_pos_files yes)
 		(dnp no)
-		(property "Reference" "#PWR0126"
+		(property "Reference" "#PWR0127"
 			(at 157.48 86.36 0)
 			(hide yes)
@@
 			(project "reflow_station"
 				(path "/77770e37-dda2-4cf3-b2f1-cea4793bc3be/68b7f722-bad3-45c2-b522-78eb1b3727cc/3afc4fe4-3fa4-4c3e-afce-f70380747f42"
-					(reference "#PWR0126")
+					(reference "#PWR0127")
 					(unit 1)
 				)
@@
 		(in_pos_files yes)
 		(dnp no)
-		(property "Reference" "#PWR0124"
+		(property "Reference" "#PWR0125"
 			(at 106.68 86.36 0)
 			(hide yes)
@@
 			(project "reflow_station"
 				(path "/77770e37-dda2-4cf3-b2f1-cea4793bc3be/68b7f722-bad3-45c2-b522-78eb1b3727cc/3afc4fe4-3fa4-4c3e-afce-f70380747f42"
-					(reference "#PWR0124")
+					(reference "#PWR0125")
 					(unit 1)
 				)
@@
 		(in_pos_files yes)
 		(dnp no)
-		(property "Reference" "#PWR0123"
+		(property "Reference" "#PWR0124"
 			(at 81.28 86.36 0)
 			(hide yes)
@@
 			(project "reflow_station"
 				(path "/77770e37-dda2-4cf3-b2f1-cea4793bc3be/68b7f722-bad3-45c2-b522-78eb1b3727cc/3afc4fe4-3fa4-4c3e-afce-f70380747f42"
-					(reference "#PWR0123")
+					(reference "#PWR0124")
 					(unit 1)
 				)
@@
 		(dnp no)
 		(fields_autoplaced yes)
-		(property "Reference" "R60"
+		(property "Reference" "R66"
 			(at 58.42 100.3299 0)
 			(show_name no)
@@
 			(project "reflow_station"
 				(path "/77770e37-dda2-4cf3-b2f1-cea4793bc3be/68b7f722-bad3-45c2-b522-78eb1b3727cc/3afc4fe4-3fa4-4c3e-afce-f70380747f42"
-					(reference "R60")
+					(reference "R66")
 					(unit 1)
 				)
@@
 		(in_pos_files yes)
 		(dnp no)
-		(property "Reference" "#PWR0122"
+		(property "Reference" "#PWR0123"
 			(at 55.88 86.36 0)
 			(hide yes)
@@
 			(project "reflow_station"
 				(path "/77770e37-dda2-4cf3-b2f1-cea4793bc3be/68b7f722-bad3-45c2-b522-78eb1b3727cc/3afc4fe4-3fa4-4c3e-afce-f70380747f42"
-					(reference "#PWR0122")
+					(reference "#PWR0123")
 					(unit 1)
 				)
@@
 		(dnp no)
 		(fields_autoplaced yes)
-		(property "Reference" "R59"
+		(property "Reference" "R65"
 			(at 246.38 87.6299 0)
 			(show_name no)
@@
 			(project "reflow_station"
 				(path "/77770e37-dda2-4cf3-b2f1-cea4793bc3be/68b7f722-bad3-45c2-b522-78eb1b3727cc/3afc4fe4-3fa4-4c3e-afce-f70380747f42"
-					(reference "R59")
+					(reference "R65")
 					(unit 1)
 				)
@@
 		(dnp no)
 		(fields_autoplaced yes)
-		(property "Reference" "R64"
+		(property "Reference" "R70"
 			(at 160.02 100.3299 0)
 			(show_name no)
@@
 			(project "reflow_station"
 				(path "/77770e37-dda2-4cf3-b2f1-cea4793bc3be/68b7f722-bad3-45c2-b522-78eb1b3727cc/3afc4fe4-3fa4-4c3e-afce-f70380747f42"
-					(reference "R64")
+					(reference "R70")
 					(unit 1)
 				)
@@
 		(dnp no)
 		(fields_autoplaced yes)
-		(property "Reference" "R63"
+		(property "Reference" "R69"
 			(at 134.62 100.3299 0)
 			(show_name no)
@@
 			(project "reflow_station"
 				(path "/77770e37-dda2-4cf3-b2f1-cea4793bc3be/68b7f722-bad3-45c2-b522-78eb1b3727cc/3afc4fe4-3fa4-4c3e-afce-f70380747f42"
-					(reference "R63")
+					(reference "R69")
 					(unit 1)
 				)
